File: Hardware/driver/input.kicad_sch (KiCad schematic)
At the start: 53 parts, among them J301 TBP01R2W-508-02BE, Q301 IXTH80N075L2, Q302 IXTH80N075L2, U301 MCP3421A2T-ECH, U302 MCP3421A1T-ECH, U303 DAC60501Z, U304 DAC60501Z, U305 DS18B20, U306 DS18B20, U307 MCP3421A3T-ECH, U308 OPA2388, U309 OPA2388

Commit message: Mostly finished routing driver board
- All traces are routed (including some big ass planes for the power
  section; these should be good to roughly 40A) and the board is
  probably good to go.

  It could use with some decorating in the bonus area though :)
Parts:
- removed F301: 20A, programmable-load:Keystone-3557-2-0, symbol Device:Fuse_Small
- added FB301: FerriteBead_Small, Inductor_SMD:L_0805_2012Metric_Pad1.05x1.20mm_HandSolder, symbol Device:FerriteBead_Small
- added TP301: VSense, TestPoint:TestPoint_Keystone_5000-5004_Miniature, symbol Connector:TestPoint
- added TP302: GND, TestPoint:TestPoint_Keystone_5000-5004_Miniature, symbol Connector:TestPoint
- J301: value TBP01R2W-508-02BE -> 1017526; footprint programmable-load:CUI_TBP01R2W-508-02BE -> programmable-load:Phoenix-TDPT-2,1017526
Connections:
- net GND: now also FB301.2, TP302.1
- net GNDPWR: now also FB301.1
- net VBUS: now also J301.2 (Pin_2)
- net VSENSE: now also TP301.1
Other:
- note added: "Connector to front panel jacks 75A max current"
- note removed: "Connector to front panel jacks Mate with TBP01P1W-508-02BE"
- note removed: "Suitable fuses: Littelfuse 0287020.H (ATOF), 0891020.NXWS (Mini) Eaton ATM-20 (Blade)"
Changed lines of the file:
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@@
+    (stroke (width 0) (type default) (color 0 0 0 0))
+  )
+  (wire (pts (xy 40.64 152.4) (xy 41.91 152.4))
     (stroke (width 0) (type default) (color 0 0 0 0))
   )
@@
   )
   (wire (pts (xy 50.8 25.4) (xy 50.8 34.29))
+    (stroke (width 0) (type default) (color 0 0 0 0))
+  )
+  (wire (pts (xy 46.99 152.4) (xy 48.26 152.4))
     (stroke (width 0) (type default) (color 0 0 0 0))
   )
@@
   )
   (text "Ringing prevention" (at 53.34 38.1 0)
-    (effects (font (size 1.27 1.27)) (justify left bottom))
-  )
-  (text "Suitable fuses: Littelfuse 0287020.H (ATOF), 0891020.NXWS (Mini)\nEaton ATM-20 (Blade)"
-    (at 217.17 163.83 0)
     (effects (font (size 1.27 1.27)) (justify left bottom))
   )
@@
     (effects (font (size 1.27 1.27)) (justify left bottom))
   )
-  (text "Connector to front panel jacks\nMate with TBP01P1W-508-02BE"
-    (at 248.92 156.21 0)
+  (text "Connector to front panel jacks\n75A max current" (at 248.92 156.21 0)
     (effects (font (size 1.27 1.27)) (justify left bottom))
   )
@@
     (pin "2")
   )
-  (symbol (lib_id "Device:Fuse_Small") (at 235.585 147.32 0) (unit 1)
-    (in_bom yes) (on_board yes) (fields_autoplaced)
-    (property "Reference" "F301" (id 0) (at 235.585 142.24 0))
-    (property "Value" "20A" (id 1) (at 235.585 144.78 0))
-    (property "Footprint" "programmable-load:Keystone-3557-2-0" (id 2) (at 235.585 147.32 0)
-      (effects (font (size 1.27 1.27)) hide)
-    )
-    (property "Datasheet" "~" (id 3) (at 235.585 147.32 0)
-      (effects (font (size 1.27 1.27)) hide)
-    )
-    (property "MPN" "3557-20" (id 4) (at 235.585 147.32 0)
-      (effects (font (size 1.27 1.27)) hide)
-    )
-    (pin "1")
-    (pin "2")
-  )
   (symbol (lib_id "Device:C_Polarized_Small") (at 215.265 102.87 0) (unit 1)
     (in_bom yes) (on_board yes) (fields_autoplaced)
@@
     (in_bom yes) (on_board yes) (fields_autoplaced)
     (property "Reference" "J301" (id 0) (at 248.92 140.97 0))
-    (property "Value" "TBP01R2W-508-02BE" (id 1) (at 248.92 143.51 0))
-    (property "Footprint" "programmable-load:CUI_TBP01R2W-508-02BE" (id 2) (at 248.92 149.86 0)
+    (property "Value" "1017526" (id 1) (at 248.92 143.51 0))
+    (property "Footprint" "programmable-load:Phoenix-TDPT-2,1017526" (id 2) (at 248.92 149.86 0)
       (effects (font (size 1.27 1.27)) hide)
     )
@@
     (pin "1")
     (pin "2")
+  )
+  (symbol (lib_id "power:GND") (at 48.26 152.4 0) (unit 1)
+    (in_bom yes) (on_board yes)
+    (property "Reference" "#PWR0350" (id 0) (at 48.26 158.75 0)
+      (effects (font (size 1.27 1.27)) hide)
+    )
+    (property "Value" "GND" (id 1) (at 48.26 156.21 0))
+    (property "Footprint" "" (id 2) (at 48.26 152.4 0)
+      (effects (font (size 1.27 1.27)) hide)
+    )
+    (property "Datasheet" "" (id 3) (at 48.26 152.4 0)
+      (effects (font (size 1.27 1.27)) hide)
+    )
+    (pin "1")
   )
   (symbol (lib_id "power:+3V3") (at 273.685 55.88 0) (mirror y) (unit 1)
@@
     )
     (property "Datasheet" "" (id 3) (at 78.74 30.48 0)
+      (effects (font (size 1.27 1.27)) hide)
+    )
+    (pin "1")
+  )
+  (symbol (lib_id "Device:FerriteBead_Small") (at 44.45 152.4 90) (unit 1)
+    (in_bom yes) (on_board yes) (fields_autoplaced)
+    (property "Reference" "FB301" (id 0) (at 44.4119 146.05 90))
+    (property "Value" "FerriteBead_Small" (id 1) (at 44.4119 148.59 90))
+    (property "Footprint" "Inductor_SMD:L_0805_2012Metric_Pad1.05x1.20mm_HandSolder" (id 2) (at 44.45 154.178 90)
+      (effects (font (size 1.27 1.27)) hide)
+    )
+    (property "Datasheet" "~" (id 3) (at 44.45 152.4 0)
+      (effects (font (size 1.27 1.27)) hide)
+    )
+    (property "MPN" "MFBM1V2012-800-R " (id 4) (at 44.45 152.4 90)
+      (effects (font (size 1.27 1.27)) hide)
+    )
+    (pin "1")
+    (pin "2")
+  )
+  (symbol (lib_id "power:GNDPWR") (at 40.64 152.4 0) (unit 1)
+    (in_bom yes) (on_board yes)
+    (property "Reference" "#PWR0310" (id 0) (at 40.64 157.48 0)
+      (effects (font (size 1.27 1.27)) hide)
+    )
+    (property "Value" "GNDPWR" (id 1) (at 40.513 156.21 0))
+    (property "Footprint" "" (id 2) (at 40.64 153.67 0)
+      (effects (font (size 1.27 1.27)) hide)
+    )
+    (property "Datasheet" "" (id 3) (at 40.64 153.67 0)
       (effects (font (size 1.27 1.27)) hide)
     )
@@
     (pin "1")
   )
+  (symbol (lib_id "Connector:TestPoint") (at 234.315 120.015 0) (mirror x) (unit 1)
+    (in_bom yes) (on_board yes) (fields_autoplaced)
+    (property "Reference" "TP301" (id 0) (at 232.41 122.0469 0)
+      (effects (font (size 1.27 1.27)) (justify right))
+    )
+    (property "Value" "VSense" (id 1) (at 232.41 124.5869 0)
+      (effects (font (size 1.27 1.27)) (justify right))
+    )
+    (property "Footprint" "TestPoint:TestPoint_Keystone_5000-5004_Miniature" (id 2) (at 239.395 120.015 0)
+      (effects (font (size 1.27 1.27)) hide)
+    )
+    (property "Datasheet" "~" (id 3) (at 239.395 120.015 0)
+      (effects (font (size 1.27 1.27)) hide)
+    )
+    (property "Color" "Yellow" (id 4) (at 234.315 120.015 0)
+      (effects (font (size 1.27 1.27)) hide)
+    )
+    (property "MPN" "5004" (id 5) (at 234.315 120.015 0)
+      (effects (font (size 1.27 1.27)) hide)
+    )
+    (pin "1")
+  )
   (symbol (lib_id "Analog_ADC:MCP3421A0T-ECH") (at 155.575 149.86 0) (mirror y) (unit 1)
     (in_bom yes) (on_board yes)
@@
     (pin "1")
   )
+  (symbol (lib_id "power:GND") (at 232.41 133.35 0) (unit 1)
+    (in_bom yes) (on_board yes) (fields_autoplaced)
+    (property "Reference" "#PWR0309" (id 0) (at 232.41 139.7 0)
+      (effects (font (size 1.27 1.27)) hide)
+    )
+    (property "Value" "GND" (id 1) (at 232.41 138.43 0))
+    (property "Footprint" "" (id 2) (at 232.41 133.35 0)
+      (effects (font (size 1.27 1.27)) hide)
+    )
+    (property "Datasheet" "" (id 3) (at 232.41 133.35 0)
+      (effects (font (size 1.27 1.27)) hide)
+    )
+    (pin "1")
+  )
   (symbol (lib_id "power:GND") (at 191.77 30.48 0) (unit 1)
     (in_bom yes) (on_board yes) (fields_autoplaced)
@@
     (pin "1")
   )
+  (symbol (lib_id "Connector:TestPoint") (at 232.41 133.35 90) (mirror x) (unit 1)
+    (in_bom yes) (on_board yes) (fields_autoplaced)
+    (property "Reference" "TP302" (id 0) (at 229.108 127 90))
+    (property "Value" "GND" (id 1) (at 229.108 129.54 90))
+    (property "Footprint" "TestPoint:TestPoint_Keystone_5000-5004_Miniature" (id 2) (at 232.41 138.43 0)
+      (effects (font (size 1.27 1.27)) hide)
+    )
+    (property "Datasheet" "~" (id 3) (at 232.41 138.43 0)
+      (effects (font (size 1.27 1.27)) hide)
+    )
+    (property "Color" "Black" (id 4) (at 232.41 133.35 0)
+      (effects (font (size 1.27 1.27)) hide)
+    )
+    (property "MPN" "5001" (id 5) (at 232.41 133.35 0)
+      (effects (font (size 1.27 1.27)) hide)
+    )
+    (pin "1")
+  )
   (symbol (lib_id "power:+3V3") (at 85.09 80.01 90) (unit 1)
     (in_bom yes) (on_board yes)
@@
     (pin "1")
   )
-  (symbol (lib_id "power:VBUS") (at 233.045 147.32 90) (unit 1)
-    (in_bom yes) (on_board yes) (fields_autoplaced)
-    (property "Reference" "#PWR0322" (id 0) (at 236.855 147.32 0)
-      (effects (font (size 1.27 1.27)) hide)
-    )
-    (property "Value" "VBUS" (id 1) (at 229.87 147.3199 90)
-      (effects (font (size 1.27 1.27)) (justify left))
-    )
-    (property "Footprint" "" (id 2) (at 233.045 147.32 0)
-      (effects (font (size 1.27 1.27)) hide)
-    )
-    (property "Datasheet" "" (id 3) (at 233.045 147.32 0)
-      (effects (font (size 1.27 1.27)) hide)
-    )
+  (symbol (lib_id "power:VBUS") (at 238.125 147.32 90) (unit 1)
+    (in_bom yes) (on_board yes) (fields_autoplaced)
+    (property "Reference" "#PWR0322" (id 0) (at 241.935 147.32 0)
+      (effects (font (size 1.27 1.27)) hide)
+    )
+    (property "Value" "VBUS" (id 1) (at 234.95 147.3199 90)
+      (effects (font (size 1.27 1.27)) (justify left))
+    )
+    (property "Footprint" "" (id 2) (at 238.125 147.32 0)
+      (effects (font (size 1.27 1.27)) hide)
+    )
+    (property "Datasheet" "" (id 3) (at 238.125 147.32 0)
+      (effects (font (size 1.27 1.27)) hide)
+    )

Commit message: Minor tweaks to layout/schematic
- Use a DC/DC to generate 5V, then generate 3V3 via an LDO from that:
  this should help filter out more of the switching noise out of the
  supplies.

  Also, this included adding a 330Ω load resistor so that the DC/DC gets
  the minimum load it expects; it burns ~15mA at 5V.

- Changes to pass DRC
Parts:
- HS301: symbol Mechanical:Heatsink_Pad_2Pin -> Mechanical:Heatsink
Changed lines of the file:
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@@
     (pin "1")
   )
-  (symbol (lib_id "programmable-load:DAC60501") (at 93.98 71.12 0) (unit 1)
+  (symbol (lib_name "DAC60501_1") (lib_id "programmable-load:DAC60501") (at 93.98 71.12 0) (unit 1)
     (in_bom yes) (on_board yes) (fields_autoplaced)
     (property "Reference" "U304" (id 0) (at 93.98 65.405 0))
@@
     (pin "10")
     (pin "2")
+    (pin "3")
     (pin "4")
     (pin "5")
@@
     (pin "7")
     (pin "8")
+    (pin "9")
   )
   (symbol (lib_id "programmable-load:OPA2388") (at 50.165 120.65 270) (unit 3)
@@
     (pin "10")
     (pin "2")
+    (pin "3")
     (pin "4")
     (pin "5")
@@
     (pin "7")
     (pin "8")
+    (pin "9")
   )
   (symbol (lib_id "power:GND") (at 174.625 59.055 0) (unit 1)
@@
     (pin "1")
   )
-  (symbol (lib_id "Mechanical:Heatsink_Pad_2Pin") (at 248.92 24.13 270) (unit 1)
+  (symbol (lib_id "Mechanical:Heatsink") (at 248.92 24.13 270) (unit 1)
     (in_bom yes) (on_board yes) (fields_autoplaced)
     (property "Reference" "HS301" (id 0) (at 252.73 22.8472 90)
@@
       (effects (font (size 1.27 1.27)) (justify left))
     )
-    (property "Footprint" "programmable-load:C40-058-AE-DUAL" (id 2) (at 247.65 24.4348 0)
-      (effects (font (size 1.27 1.27)) hide)
-    )
-    (property "Datasheet" "~" (id 3) (at 247.65 24.4348 0)
+    (property "Footprint" "programmable-load:C40-058-AE-DUAL" (id 2) (at 248.92 24.4348 0)
+      (effects (font (size 1.27 1.27)) hide)
+    )
+    (property "Datasheet" "~" (id 3) (at 248.92 24.4348 0)
       (effects (font (size 1.27 1.27)) hide)
     )
@@
       (effects (font (size 1.27 1.27)) hide)
     )
-    (pin "1")
-    (pin "2")
   )
   (symbol (lib_id "power:GNDPWR") (at 266.065 127.635 0) (unit 1)

Commit message: Fixed some part numbers in schematic
- Also updated some of the annotations, they were out-of-date with
  respect to what the current status was
Parts:
- R306, R309, R313, R314, R315: value 5k -> 4k99
- U303, U304: MPN (none) -> DAC60501ZDGSR
- U308, U309: MPN (none) -> OPA2388IDR
Other:
- note added: "Clips: CLA-T247-21E (TO-247) Insulator: Bergquist SP900S-0.009-00-104"
- note removed: "Clips: CLA-T247-21E (TO-247)"
Changed lines of the file:
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@@
     (effects (font (size 1.27 1.27)) (justify left bottom))
   )
-  (text "Clips: CLA-T247-21E (TO-247)" (at 247.65 31.75 0)
+  (text "Clips: CLA-T247-21E (TO-247)\nInsulator: Bergquist SP900S-0.009-00-104"
+    (at 240.03 33.02 0)
     (effects (font (size 1.27 1.27)) (justify left bottom))
   )
@@
       (effects (font (size 1.27 1.27)) hide)
     )
+    (property "MPN" "OPA2388IDR" (id 4) (at 64.77 25.4 0)
+      (effects (font (size 1.27 1.27)) hide)
+    )
     (pin "1")
     (pin "2")
@@
       (effects (font (size 1.27 1.27)) (justify right))
     )
-    (property "Value" "5k" (id 1) (at 57.15 52.0699 0)
+    (property "Value" "4k99" (id 1) (at 57.15 52.0699 0)
       (effects (font (size 1.27 1.27)) (justify right))
     )
@@
       (effects (font (size 1.27 1.27)) hide)
     )
+    (property "MPN" "OPA2388IDR" (id 4) (at 177.8 25.4 0)
+      (effects (font (size 1.27 1.27)) hide)
+    )
     (pin "1")
     (pin "2")
@@
       (effects (font (size 1.27 1.27)) hide)
     )
+    (property "MPN" "OPA2388IDR" (id 4) (at 101.6 25.4 0)
+      (effects (font (size 1.27 1.27)) hide)
+    )
     (pin "5")
     (pin "6")
@@
     )
     (property "Datasheet" "https://www.ti.com/lit/ds/symlink/dac60501.pdf" (id 3) (at 93.98 64.77 0)
+      (effects (font (size 1.27 1.27)) hide)
+    )
+    (property "MPN" "DAC60501ZDGSR" (id 4) (at 93.98 71.12 0)
       (effects (font (size 1.27 1.27)) hide)
     )
@@
       (effects (font (size 1.27 1.27)) (justify left))
     )
-    (property "Value" "5k" (id 1) (at 170.18 52.0699 0)
+    (property "Value" "4k99" (id 1) (at 170.18 52.0699 0)
       (effects (font (size 1.27 1.27)) (justify left))
     )
@@
     (in_bom yes) (on_board yes)
     (property "Reference" "R309" (id 0) (at 246.38 114.935 90))
-    (property "Value" "5k" (id 1) (at 246.38 117.475 90))
+    (property "Value" "4k99" (id 1) (at 246.38 117.475 90))
     (property "Footprint" "Resistor_SMD:R_0805_2012Metric_Pad1.20x1.40mm_HandSolder" (id 2) (at 246.38 120.015 0)
       (effects (font (size 1.27 1.27)) hide)
@@
     (in_bom yes) (on_board yes)
     (property "Reference" "R313" (id 0) (at 194.31 17.78 90))
-    (property "Value" "5k" (id 1) (at 194.31 20.32 90))
+    (property "Value" "4k99" (id 1) (at 194.31 20.32 90))
     (property "Footprint" "Resistor_SMD:R_0805_2012Metric_Pad1.20x1.40mm_HandSolder" (id 2) (at 194.31 22.86 0)
       (effects (font (size 1.27 1.27)) hide)
@@
     )
     (property "Datasheet" "https://www.ti.com/lit/ds/symlink/dac60501.pdf" (id 3) (at 208.28 62.23 0)
+      (effects (font (size 1.27 1.27)) hide)
+    )
+    (property "MPN" "DAC60501ZDGSR" (id 4) (at 208.28 68.58 0)
       (effects (font (size 1.27 1.27)) hide)
     )
@@
     (in_bom yes) (on_board yes)
     (property "Reference" "R306" (id 0) (at 81.28 17.78 90))
-    (property "Value" "5k" (id 1) (at 81.28 20.32 90))
+    (property "Value" "4k99" (id 1) (at 81.28 20.32 90))
     (property "Footprint" "Resistor_SMD:R_0805_2012Metric_Pad1.20x1.40mm_HandSolder" (id 2) (at 81.28 22.86 0)
       (effects (font (size 1.27 1.27)) hide)
