File: Hardware/driver/trigger.kicad_sch (KiCad schematic)
At the start: 11 parts, among them J501 Conn_Coaxial, U501 FODM217B, U502 74LVC1G17

Commit message: Start work on remote VSense; driver board tweaks
- Use the DAC reference as the positive end of the null adjustment
  trimmers, rather than the +3V3 supply; this should make the adjustment
  actually useful and persistent rather than relying on the relationship
  between the 3V3 rail and the DAC's internal reference.

- Moved the 1Wire controller slightly to allow relocating the zero
  offset trimmer for the first channel

- Start work on remote VSense

  This works by selecting between either voltage sensing at the source
  terminals, or an external sense input connected to another set of
  terminals. These are switched by a latching relay (as to provide
  satisfying clicky noises) and then go into an op amp working as a
  differential amplifier; it performs a 50:1 gain (obviating the need
  for resistor dividers, and providing greater accuracy) and that then
  goes into the measurement ADC as normal.

  We have to still figure out how to drive the relay (probably just an
  IO expander?) and place those components on the board.
Parts:
- renumbered C502 to C501, C501 to C502, R503 to R501, R501 to R503, U502 to U501, U501 to U502
Changed lines of the file:
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@@
   (symbol (lib_id "74xGxx:74LVC1G17") (at 176.53 36.83 0) (mirror y) (unit 1)
     (in_bom yes) (on_board yes) (fields_autoplaced)
-    (property "Reference" "U502" (id 0) (at 177.165 29.21 0))
+    (property "Reference" "U501" (id 0) (at 177.165 29.21 0))
     (property "Value" "74LVC1G17" (id 1) (at 177.165 31.75 0))
     (property "Footprint" "Package_TO_SOT_SMD:SOT-23-5_HandSoldering" (id 2) (at 176.53 36.83 0)
@@
   (symbol (lib_id "Device:C_Small") (at 212.725 36.83 90) (unit 1)
     (in_bom yes) (on_board yes) (fields_autoplaced)
-    (property "Reference" "C501" (id 0) (at 212.7313 29.845 90))
+    (property "Reference" "C502" (id 0) (at 212.7313 29.845 90))
     (property "Value" "1µF" (id 1) (at 212.7313 32.385 90))
     (property "Footprint" "Capacitor_SMD:C_0805_2012Metric_Pad1.18x1.45mm_HandSolder" (id 2) (at 212.725 36.83 0)
@@
   (symbol (lib_id "Device:R_Small") (at 257.175 31.75 90) (unit 1)
     (in_bom yes) (on_board yes)
-    (property "Reference" "R501" (id 0) (at 257.175 26.67 90))
+    (property "Reference" "R503" (id 0) (at 257.175 26.67 90))
     (property "Value" "100R" (id 1) (at 257.175 29.21 90))
     (property "Footprint" "Resistor_SMD:R_0805_2012Metric_Pad1.20x1.40mm_HandSolder" (id 2) (at 257.175 31.75 0)
@@
   (symbol (lib_id "Isolator:FODM217B") (at 238.76 34.29 0) (mirror y) (unit 1)
     (in_bom yes) (on_board yes) (fields_autoplaced)
-    (property "Reference" "U501" (id 0) (at 238.76 25.4 0))
+    (property "Reference" "U502" (id 0) (at 238.76 25.4 0))
     (property "Value" "FODM217B" (id 1) (at 238.76 27.94 0))
     (property "Footprint" "Package_SO:SOP-4_4.4x2.6mm_P1.27mm" (id 2) (at 238.76 40.64 0)
@@
   (symbol (lib_id "Device:C_Small") (at 176.53 56.515 0) (mirror y) (unit 1)
     (in_bom yes) (on_board yes) (fields_autoplaced)
-    (property "Reference" "C502" (id 0) (at 173.99 55.2512 0)
+    (property "Reference" "C501" (id 0) (at 173.99 55.2512 0)
       (effects (font (size 1.27 1.27)) (justify left))
     )
@@
   (symbol (lib_id "power:+3V3") (at 231.14 31.75 90) (unit 1)
     (in_bom yes) (on_board yes) (fields_autoplaced)
-    (property "Reference" "#PWR0127" (id 0) (at 234.95 31.75 0)
+    (property "Reference" "#PWR0507" (id 0) (at 234.95 31.75 0)
       (effects (font (size 1.27 1.27)) hide)
     )
@@
   (symbol (lib_id "power:GND") (at 199.39 45.72 0) (unit 1)
     (in_bom yes) (on_board yes) (fields_autoplaced)
-    (property "Reference" "#PWR0128" (id 0) (at 199.39 52.07 0)
+    (property "Reference" "#PWR0506" (id 0) (at 199.39 52.07 0)
       (effects (font (size 1.27 1.27)) hide)
     )
@@
   (symbol (lib_id "Device:R_Small") (at 158.75 44.45 180) (unit 1)
     (in_bom yes) (on_board yes) (fields_autoplaced)
-    (property "Reference" "R503" (id 0) (at 160.655 43.1799 0)
-      (effects (font (size 1.27 1.27)) (justify right))
-    )
+    (property "Reference" "R501" (id 0) (at 160.655 43.1799 0)
+      (effects (font (size 1.27 1.27)) (justify right))
+    )

Commit message: Add some missing part numbers to analog board
- Some components on analog load were missing part numbers, so this adds
  them. It also fixes a few components with the same value, where some
  had a part number and others didn't.
Parts:
- C502: value 1µF -> (none); footprint Capacitor_SMD:C_0805_2012Metric_Pad1.18x1.45mm_HandSolder -> (none); MPN 187-CL21B105KBFNNNG -> CL21B105KBFNNNG
- R501: value 10k -> (none); footprint Resistor_SMD:R_0805_2012Metric_Pad1.20x1.40mm_HandSolder -> (none); MPN (none) -> RMC1/10-103JTP
Changed lines of the file:
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@@
     (in_bom yes) (on_board yes) (fields_autoplaced)
     (property "Reference" "C502" (id 0) (at 212.7313 29.845 90))
-    (property "Value" "1µF" (id 1) (at 212.7313 32.385 90))
-    (property "Footprint" "Capacitor_SMD:C_0805_2012Metric_Pad1.18x1.45mm_HandSolder" (id 2) (at 212.725 36.83 0)
+    (property "Value" "" (id 1) (at 212.7313 32.385 90))
+    (property "Footprint" "" (id 2) (at 212.725 36.83 0)
       (effects (font (size 1.27 1.27)) hide)
     )
@@
       (effects (font (size 1.27 1.27)) hide)
     )
-    (property "MPN" "187-CL21B105KBFNNNG" (id 4) (at 212.725 36.83 0)
+    (property "MPN" "CL21B105KBFNNNG" (id 4) (at 212.725 36.83 0)
       (effects (font (size 1.27 1.27)) hide)
     )
@@
       (effects (font (size 1.27 1.27)) (justify right))
     )
-    (property "Value" "10k" (id 1) (at 160.655 45.7199 0)
-      (effects (font (size 1.27 1.27)) (justify right))
-    )
-    (property "Footprint" "Resistor_SMD:R_0805_2012Metric_Pad1.20x1.40mm_HandSolder" (id 2) (at 158.75 44.45 0)
+    (property "Value" "" (id 1) (at 160.655 45.7199 0)
+      (effects (font (size 1.27 1.27)) (justify right))
+    )
+    (property "Footprint" "" (id 2) (at 158.75 44.45 0)
       (effects (font (size 1.27 1.27)) hide)
     )
@@
       (effects (font (size 1.27 1.27)) hide)
     )
+    (property "MPN" "RMC1/10-103JTP" (id 4) (at 158.75 44.45 0)
+      (effects (font (size 1.27 1.27)) hide)
+    )
