File: Hardware/front-bonus-display/front-bonus-display.kicad_sch (KiCad schematic)
At the start: 11 parts, among them J101 Conn_02x05_Odd_Even, U101 AT24CS32-SSHM

Commit message: Finish routing of bonus display
- Completed layout and routing of the bonus display; this is just the
  LED driver (with discrete transistors for each of the three possible
  cathode channels, and associated current limiting resistors)

- Added an improved TO-247 dual pin footprint with larger holes for the
  power resistors to be used on the analog board
Parts:
- added C105: 100nF, Capacitor_SMD:C_0805_2012Metric_Pad1.18x1.45mm_HandSolder, symbol Device:C_Small
- added JP102: Jumper_3_Open, Connector_PinHeader_2.54mm:PinHeader_1x03_P2.54mm_Vertical, symbol Connector_Generic:Conn_01x03
- added Q101, Q102, Q103: MMBT3904, Package_TO_SOT_SMD:SOT-323_SC-70_Handsoldering, symbol Transistor_BJT:MMBT3904
- added R101: 27R, Resistor_SMD:R_0805_2012Metric_Pad1.20x1.40mm_HandSolder, symbol Device:R_Small
- added R102: 10R, Resistor_SMD:R_0805_2012Metric_Pad1.20x1.40mm_HandSolder, symbol Device:R_Small
- added R103: 20R, Resistor_SMD:R_0805_2012Metric_Pad1.20x1.40mm_HandSolder, symbol Device:R_Small
- added R104, R105, R106: 10k, Resistor_SMD:R_0805_2012Metric_Pad1.20x1.40mm_HandSolder, symbol Device:R_Small
- added U102: PCA9633, Package_SO:TSSOP-16_4.4x5mm_P0.65mm, symbol programmable-load:PCA9633
- C102: value (none) -> 1µF; footprint (none) -> Capacitor_SMD:C_0805_2012Metric_Pad1.18x1.45mm_HandSolder
- JP101: value (none) -> Cfg WP; footprint (none) -> Jumper:SolderJumper-3_P1.3mm_Bridged12_RoundedPad1.0x1.5mm_NumberLabels
Connections:
- net I²C_SCL is gone; now on net I2C_SCL: DS101.17 (SCLK)
- net +3V3: now also DS101.1 (A1/AGR/AERW), C105.1, JP102.3 (Pin_3), U102.1 (A0), U102.14 (A5), U102.15 (A6), U102.16 (VCC)
- net GND: now also C105.2, Q101.2 (E), Q102.2 (E), Q103.2 (E), R104.1, R105.1, R106.1, U102.10 (~{OE}), U102.11 (A4), U102.2 (A1), U102.7 (A2), U102.8 (A3), U102.9 (GND)
- net I2C_SCL: now also J101.5 (Pin_5), U102.12 (SCL)
- net I2C_SDA: now also J101.7 (Pin_7), U102.13 (SDA)
- net ~{RESET}: now also J101.9 (Pin_9)
- net at DS101.10 (A2/NC/CW): now also JP102.2 (Pin_2)
- net at DS101.2 (C1/CR/CR): now also R101.2
- net at DS101.9 (C2/CG/CE): now also R103.2
- net ~{IRQ}: now reaches J101.8 (Pin_8)
- new net: JP102.1 (Pin_1), R102.2
- new net: Q102.1 (B), R105.2, U102.4 (LED1)
- new net: Q101.1 (B), R104.2, U102.3 (LED0)
- new net: Q103.1 (B), R106.2, U102.5 (LED2)
- new net LED_C1: Q103.3 (C), R101.1
- new net LED_C2: Q102.3 (C), R102.1
- new net LED_C3: Q101.3 (C), R103.1
- no-connect marks 0 -> 1
Other:
- note added: "Backlight Driver"
- note added: "Resistors are set for -GR backlight JP102: set 2-3 for amber backlight set 1-2 for GR or GRW backlights"
