File: Hardware/analog/power.kicad_sch (KiCad schematic)
At the start: 34 parts

Commit message: Temperature sensing & cleanup for analog board
- Added the auxiliary temperature sensing ADC, and routed it to the
  analog temperature sensors on the front and rear of the MOSFET
  heatsink

- Added an LM75 sensor to measure the analog board ambient temperature
  (for better temperature control/fan control)

  This may end up being a DNP item if it's not really useful or
  otherwise necessary.

- Fixes to a few symbols (namely pin directions) to pass ERC
Changed lines of the file:
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@@
   (junction (at 133.35 75.565) (diameter 0) (color 0 0 0 0)
   )
-  (junction (at 81.28 61.595) (diameter 0) (color 0 0 0 0)
-  )
   (junction (at 66.04 94.615) (diameter 0) (color 0 0 0 0)
   )
@@
   (junction (at 278.765 114.3) (diameter 0) (color 0 0 0 0)
   )
-  (junction (at 81.28 31.75) (diameter 0) (color 0 0 0 0)
-  )
   (junction (at 149.225 75.565) (diameter 0) (color 0 0 0 0)
   )
@@
   (junction (at 160.02 65.405) (diameter 0) (color 0 0 0 0)
   )
-  (junction (at 168.275 31.75) (diameter 0) (color 0 0 0 0)
-  )
   (junction (at 93.98 94.615) (diameter 0) (color 0 0 0 0)
   )
@@
   )
   (junction (at 278.765 128.905) (diameter 0) (color 0 0 0 0)
+  )
+  (junction (at 140.335 88.265) (diameter 0) (color 0 0 0 0)
   )
   (junction (at 34.925 31.75) (diameter 0) (color 0 0 0 0)
@@
     (pin "2")
   )
-  (symbol (lib_id "power:PWR_FLAG") (at 167.64 65.405 270) (mirror x) (unit 1)
-    (in_bom yes) (on_board yes)
-    (default_instance (reference "U") (unit 1) (value "") (footprint ""))
-    (property "Reference" "U" (id 0) (at 169.545 65.405 0)
-      (effects (font (size 1.27 1.27)) hide)
-    )
-    (property "Value" "" (id 1) (at 170.815 65.405 90)
-      (effects (font (size 1.27 1.27)) (justify left))
-    )
-    (property "Footprint" "" (id 2) (at 167.64 65.405 0)
-      (effects (font (size 1.27 1.27)) hide)
-    )
-    (property "Datasheet" "~" (id 3) (at 167.64 65.405 0)
-      (effects (font (size 1.27 1.27)) hide)
-    )
-    (pin "1")
-  )
   (symbol (lib_id "Device:R_Small") (at 266.7 144.145 90) (unit 1)
     (in_bom yes) (on_board yes)
@@
     )
     (property "Datasheet" "" (id 3) (at 46.355 69.215 0)
-      (effects (font (size 1.27 1.27)) hide)
-    )
-    (pin "1")
-  )
-  (symbol (lib_id "power:PWR_FLAG") (at 81.28 31.75 270) (mirror x) (unit 1)
-    (in_bom yes) (on_board yes) (fields_autoplaced)
-    (default_instance (reference "U") (unit 1) (value "") (footprint ""))
-    (property "Reference" "U" (id 0) (at 83.185 31.75 0)
-      (effects (font (size 1.27 1.27)) hide)
-    )
-    (property "Value" "" (id 1) (at 84.455 31.7499 90)
-      (effects (font (size 1.27 1.27)) (justify left))
-    )
-    (property "Footprint" "" (id 2) (at 81.28 31.75 0)
-      (effects (font (size 1.27 1.27)) hide)
-    )
-    (property "Datasheet" "~" (id 3) (at 81.28 31.75 0)
       (effects (font (size 1.27 1.27)) hide)
     )
@@
     (pin "1")
   )
-  (symbol (lib_id "power:PWR_FLAG") (at 168.275 31.75 270) (mirror x) (unit 1)
-    (in_bom yes) (on_board yes)
-    (default_instance (reference "U") (unit 1) (value "") (footprint ""))
-    (property "Reference" "U" (id 0) (at 170.18 31.75 0)
-      (effects (font (size 1.27 1.27)) hide)
-    )
-    (property "Value" "" (id 1) (at 171.45 31.75 90)
-      (effects (font (size 1.27 1.27)) (justify left))
-    )
-    (property "Footprint" "" (id 2) (at 168.275 31.75 0)
-      (effects (font (size 1.27 1.27)) hide)
-    )
-    (property "Datasheet" "~" (id 3) (at 168.275 31.75 0)
-      (effects (font (size 1.27 1.27)) hide)
-    )
-    (pin "1")
-  )
   (symbol (lib_id "power:+15V") (at 26.67 61.595 90) (mirror x) (unit 1)
     (in_bom yes) (on_board yes) (fields_autoplaced)
@@
     )
     (property "Datasheet" "" (id 3) (at 264.16 114.3 0)
+      (effects (font (size 1.27 1.27)) hide)
+    )
+    (pin "1")
+  )
+  (symbol (lib_id "power:PWR_FLAG") (at 140.335 88.265 0) (unit 1)
+    (in_bom yes) (on_board yes) (fields_autoplaced)
+    (default_instance (reference "#FLG") (unit 1) (value "PWR_FLAG") (footprint ""))
+    (property "Reference" "#FLG" (id 0) (at 140.335 86.36 0)
+      (effects (font (size 1.27 1.27)) hide)
+    )
+    (property "Value" "PWR_FLAG" (id 1) (at 140.335 85.09 0)
+      (effects (font (size 1.27 1.27)) hide)
+    )
+    (property "Footprint" "" (id 2) (at 140.335 88.265 0)
+      (effects (font (size 1.27 1.27)) hide)
+    )
+    (property "Datasheet" "~" (id 3) (at 140.335 88.265 0)
       (effects (font (size 1.27 1.27)) hide)
     )
@@
       (effects (font (size 1.27 1.27)) hide)
     )
-    (pin "1")
-  )
-  (symbol (lib_id "power:PWR_FLAG") (at 81.28 61.595 270) (mirror x) (unit 1)
-    (in_bom yes) (on_board yes) (fields_autoplaced)
-    (default_instance (reference "U") (unit 1) (value "") (footprint ""))
-    (property "Reference" "U" (id 0) (at 83.185 61.595 0)
-      (effects (font (size 1.27 1.27)) hide)
-    )
-    (property "Value" "" (id 1) (at 84.455 61.5949 90)
-      (effects (font (size 1.27 1.27)) (justify left))
-    )
-    (property "Footprint" "" (id 2) (at 81.28 61.595 0)
-      (effects (font (size 1.27 1.27)) hide)
-    )
-    (property "Datasheet" "~" (id 3) (at 81.28 61.595 0)
-      (effects (font (size 1.27 1.27)) hide)
-    )
