File: Hardware/rear/rear.kicad_sch (KiCad schematic)
At the start: 18 parts, among them J101 Conn_02x10_Odd_Even, J102 USB_B, J103 ARJC07-111071A, U101 AT24CS32-SSHM, U102 WE-TVS-82400102, U103 MCP3021

Commit message: Re-design around STM32MP1 (#2)
* Start work on rev3 hardware

- This fits the Technomet R110 enclosure and supports multiple load
  boards, connected via CAN rather than I2C. Each load has a
  microcontroller of its own.

* More new layout stuff

- More work on the new controller board layout

- Rework rear IO board for the new Technomet rear panel (it has an
  expansion connector for CAN also, and features four screw holes
  instead of two)

- Added a few footprints (expansion RJ45 connector; some
  horizontal/vertical headers)

* Work on controller VSense, power

- Routed 3V3 switching supply

- Created footprint and symbols for Kemet EA2 series latching relay

- Added relays to controller to handle routing of voltage sense inputs
  to the sampling ADC

* Rear IO rework

- Mostly finished the rear IO board rework (adding the CAN filtering and
  switchable termination; trigger input pulse shaper; fuses for
  expansion +12V)

- Changed encoder type on front panel for a shorter type

- Created schematic models and footprints for Bournds DR311 chokes;
  Mill-Max 2108 solder turrets

* More work on new controller board

- Switched mains connection for a push-in screw terminal, rather than a
  pluggable block (takes up less space, less parts)

- Added input terminal for rear VSense inputs

- Added -5V supply (same circuit as on analog board; required for
  voltage input sense)

- Replaced beeper with a side-firing version. It takes up a bunch less
  space vertically, and also now added a resistor to (hopefully) make it
  somewhat more quiet

- Added connector for bonus displays

* Add "bonus display" board

- Created the bonus display board, which houses a chip-on-glass 4x10
  text character display. It's meant to be mounted next to the input
  jacks to show a constant location of current/voltage, even if the main
  display is used for menus or other stuff.

- More tweaks to controller board, to do with power g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
Parts:
- removed J101: Conn_02x10_Odd_Even, Connector_PinHeader_1.27mm:PinHeader_2x10_P1.27mm_Vertical_SMD, symbol Connector_Generic:Conn_02x10_Odd_Even
- removed U103: MCP3021, Package_TO_SOT_SMD:SOT-23-5_HandSoldering, symbol programmable-load:MCP3021
- added C106: 100nF, Capacitor_SMD:C_0805_2012Metric_Pad1.18x1.45mm_HandSolder, symbol Device:C_Small
- added D101, D102: Green, LED_SMD:LED_0805_2012Metric_Pad1.15x1.40mm_HandSolder, symbol Device:LED_Small
- added D103: ESDONCAN1, Package_TO_SOT_SMD:SOT-23_Handsoldering, symbol Device:D_TVS_Dual_AAC
- added D104: Panjit SS14, Diode_SMD:D_SMA_Handsoldering, symbol Device:D_Schottky_Small
- added D105: 1N4148W, Diode_SMD:D_SOD-123, symbol Diode:1N4148W
- added F101: 500mA, Fuse:Fuse_1206_3216Metric_Pad1.42x1.75mm_HandSolder, symbol Device:Polyfuse_Small
- added FB101: FerriteBead_Small, Inductor_SMD:L_0805_2012Metric_Pad1.05x1.20mm_HandSolder, symbol Device:FerriteBead_Small
- added H103, H104: MountingHole, MountingHole:MountingHole_2.7mm_M2.5, symbol Mechanical:MountingHole
- added J101: Conn_02x10_Odd_Even, Connector_PinHeader_1.27mm:PinHeader_2x13_P1.27mm_Vertical, symbol Connector_Generic:Conn_02x13_Odd_Even
- added J104: CRJ061-L1-TH, programmable-load:CUI_CRJ061-L1-TH, symbol programmable-load:CRJ061-L1-TH
- added J105: (no value), symbol Connector_Generic:Conn_01x01
- added J106: Conn_01x01, programmable-load:MillMax-2108-2, symbol Connector_Generic:Conn_01x01
- added L101: DR331-513BE, programmable-load:Bourns-DR331-0-0-MFG, symbol Device:L_Ferrite_Coupled_1423
- added R105, R106, R107: 1k, Resistor_SMD:R_0805_2012Metric_Pad1.20x1.40mm_HandSolder, symbol Device:R_Small
- added R108, R109: (no value), symbol Device:R_Small
- added R110: 47k, Resistor_SMD:R_0805_2012Metric_Pad1.20x1.40mm_HandSolder, symbol Device:R_Small
- added RV101: 500k, programmable-load:Potentiometer_Nidec_Copal_CT94EW, symbol Device:R_Potentiometer_Trim
- added TP101: Trigger, TestPoint:TestPoint_Keystone_5000-5004_Miniature, symbol Connector:TestPoint
- added U103: XRA1200, Package_SO:TSSOP-16_4.4x5mm_P0.65mm, symbol programmable-load:XRA1200
- added U104: (no value), symbol programmable-load:TLP170A
- added U105: FODM217B, Package_SO:SOP-4_4.4x2.6mm_P1.27mm, symbol Isolator:FODM217B
- added U106: 74LVC1G17, Package_TO_SOT_SMD:SOT-23-5_HandSoldering, symbol 74xGxx:74LVC1G17
- C102: value 100nF -> (none); footprint Capacitor_SMD:C_0805_2012Metric_Pad1.18x1.45mm_HandSolder -> (none); MPN CL21B104KACNFNC -> CL21B105KBFNNNG
- R103: value 7k5 -> 100R; MPN WR08X752 JTL -> WR08X101 JTL
- R104: value 12k -> 100R; MPN RMC1/10-123JTP -> WR08X101 JTL
Connections:
- net +3V3: now also R103.2, R104.2, C106.1, J101.10 (Pin_10), J101.12 (Pin_12), R105.1, R106.1, U103.16 (VCC), U105.4, U106.5 (VCC); no longer C102.1
- net ETH_LED0: now also J101.11 (Pin_11)
- net ETH_LED1: now also J101.9 (Pin_9)
- net ETH_RX+: now also J101.26 (Pin_26)
- net ETH_RX-: now also J101.24 (Pin_24)
- net ETH_TX+: now also J101.25 (Pin_25)
- net ETH_TX-: now also J101.23 (Pin_23)
- net GND: now also C106.2, D103.3 (common), J101.13 (Pin_13), J101.14 (Pin_14), J101.17 (Pin_17), J101.2 (Pin_2), J101.21 (Pin_21), J101.22 (Pin_22), J101.4 (Pin_4), J101.6 (Pin_6), J104.7, J104.8, R110.1, RV101.1, RV101.2, U103.1 (A0), U103.2 (A1), U103.3 (A2), U103.8 (GND), U104.3, U106.3 (GND); no longer C102.2, R104.2
- net SCL: now also J101.8 (Pin_8), U103.14 (SCL)
- net SDA: now also J101.5 (Pin_5), U103.15 (SDA)
- net USB_D+: now also J101.1 (Pin_1)
- net USB_D-: now also J101.3 (Pin_3)
- net VBUS: no longer R103.1
- net ~{IRQ}: now also J101.7 (Pin_7), U103.13 (~{IRQ})
- net at R104.1: now also J104.12; no longer R103.2
- new net: D103.1 (A1), J104.2, L101.1
- new net: D103.2 (A2), J104.1, L101.2
- new net: R108.1, U104.6
- new net: D105.1 (K), R109.1, U105.1
- new net: D105.2 (A), J106.1 (Pin_1), U105.2
- new net: C102.1, RV101.3, TP101.1, U106.2
- new net: D101.2 (A), R105.2
- new net: J105.1 (Pin_1), R109.2
- new net: J104.10, R103.1
- new net: F101.1, FB101.2
- new net: D104.1 (K), F101.2
- new net: R107.1, U104.1
- new net: FB101.1, J104.4, J104.5
- new net: D102.2 (A), R106.2
- new net: C102.2, R110.2, U105.3
- new net +12V: D104.2 (A), J101.15 (Pin_15), J101.16 (Pin_16)
- new net CANH: J101.20 (Pin_20), L101.3, R108.2
- new net CANL: J101.18 (Pin_18), L101.4, U104.4
- new net TERM_EN: R107.2, U103.12 (P7)
- new net TRIGGER: J101.19 (Pin_19), U106.4
- new net ~{EXT_LED0}: J104.9, U103.7 (P3)
- new net ~{EXT_LED1}: J104.11, U103.6 (P2)
- new net ~{LED_TRIGGER}: D102.1 (K), U103.4 (P0)
- new net ~{LED_VSENSE}: D101.1 (K), U103.5 (P1)
- no-connect marks 3 -> 10
Other:
- note added: "CAN Termination"
- note added: "Expansion"
- note added: "External Trigger"
- note added: "IO Expander"
- note added: "Indicators"
- note added: "I²C address: 0b0100000"
- note removed: "I²C address: 0b1001000"
- note removed: "There is absolutely no reason this needs to be an ADC other than it was cheaper and smaller than an I2C GPIO expander for a single IO line lol"
- note removed: "VBUS Sensing"
- title: Rear IO (USB + Ethernet) -> Rear IO
- moved on the sheet: C101, H101, H102
