File: Hardware/controller/canbus.kicad_sch (KiCad schematic)
At the start: 11 parts

Commit message: ERC and manufacturability tweaks for controller
- Fixed issues that prevented successful ERC runs from happening

- Tweaked a few routing/traces, mostly to increase some clearances and
  spacings

- Added an LM75-style ambient temperature sensor
Other:
- note removed: "TODO: add CAN transceiver"
Changed lines of the file:
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@@
     (effects (font (size 2.54 2.54)) (justify left bottom))
-  )
-  (text "TODO: add CAN transceiver" (at 88.265 31.75 0)
-    (effects (font (size 1.27 1.27)) (justify left bottom))
   )
   (text "CAN Transceiver" (at 82.55 19.05 0)

Commit message: hw: start working on rev4 controller
- removed SPI for display, and the associated SPI mux nonsense, and any
  superfluous resistors for pull-ups

- removed MAC address EEPROM

- start adding i2c RTC (which will also contain EEPROM with the MAC of
  the system, lol)

- start moving some components from bottom to top side of board

- tweaked positions of some mains voltage traces

- increased values of power indicator LED's current dropping resistors

- take 3V3 from SoM rather than generate it ourselves
Other:
- title: (none) -> Programmable Load Controller
Changed lines of the file:
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@@
 (kicad_sch (version 20220404) (generator eeschema)
   (paper "A4")
+  (title_block
+    (title "Programmable Load Controller")
+    (date "2022-06-28")
+    (rev "4")
+  )
   (junction (at 21.59 139.7) (diameter 0) (color 0 0 0 0)
   )

Commit message: hw: add more part numbers, cleanup
- Added JLCPCB part numbers for more passive components

- Added a status LED for the rear of the board (next to the device USB
  port)
Parts:
- C: JLCPCB (none) -> C1644
- U: JLCPCB (none) -> C14663
- U: JLCPCB (none) -> C25804
- U: JLCPCB (none) -> C7171
- Y: JLCPCB (none) -> C13738
Changed lines of the file:
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@@
+      (effects (font (size 1.27 1.27)) hide)
+    )
+    (property "JLCPCB" "C14663" (id 5) (at 57.15 76.2 0)
       (effects (font (size 1.27 1.27)) hide)
     )
@@
       (effects (font (size 1.27 1.27)) hide)
     )
+    (property "JLCPCB" "C13738" (id 5) (at 25.4 72.39 0)
+      (effects (font (size 1.27 1.27)) hide)
+    )
     (pin "1")
     (pin "2")
@@
       (effects (font (size 1.27 1.27)) hide)
     )
+    (property "JLCPCB" "C25804" (id 5) (at 25.4 139.7 90)
+      (effects (font (size 1.27 1.27)) hide)
+    )
     (pin "1")
     (pin "2")
@@
       (effects (font (size 1.27 1.27)) hide)
     )
+    (property "JLCPCB" "C14663" (id 5) (at 101.6 73.025 0)
+      (effects (font (size 1.27 1.27)) hide)
+    )
     (pin "1")
     (pin "2")
@@
     )
     (property "Datasheet" "~" (id 3) (at 22.86 84.455 0)
+      (effects (font (size 1.27 1.27)) hide)
+    )
+    (property "JLCPCB" "C1644" (id 4) (at 22.86 84.455 0)
       (effects (font (size 1.27 1.27)) hide)
     )
@@
       (effects (font (size 1.27 1.27)) hide)
     )
+    (property "JLCPCB" "C14663" (id 5) (at 127 73.025 0)
+      (effects (font (size 1.27 1.27)) hide)
+    )
     (pin "1")
     (pin "2")
@@
       (effects (font (size 1.27 1.27)) hide)
     )
+    (property "JLCPCB" "C1644" (id 4) (at 27.94 84.455 0)
+      (effects (font (size 1.27 1.27)) hide)
+    )
     (pin "1")
     (pin "2")
@@
       (effects (font (size 1.27 1.27)) hide)
     )
+    (property "JLCPCB" "C7171" (id 5) (at 116.205 73.025 0)
+      (effects (font (size 1.27 1.27)) hide)
+    )
     (pin "1")
     (pin "2")
@@
       (effects (font (size 1.27 1.27)) hide)
     )
+    (property "JLCPCB" "C25804" (id 5) (at 25.4 149.225 90)
+      (effects (font (size 1.27 1.27)) hide)
+    )
