File: Hardware/controller/io-rear.kicad_sch (KiCad schematic)
At the start: 40 parts

Commit message: Minor tweaks to main controller board
- Add SoM reset switch

- Add LED to indicate when expansion power is enabled

- Add labels for most connectors to the outside world, including a
  pinout for the expansion terminals

- Minor rearrangement of some passives
Parts:
- added U: (no value), symbol Device:LED_Small
- added U: (no value), symbol Device:R_Small
Connections:
- net GND: now also U.1 (K)
- net at K.5, U.2 (A): now also U.2
- new net: U.1, U.2 (A)
Changed lines of the file:
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@@
   (junction (at 113.03 50.165) (diameter 0) (color 0 0 0 0)
+  )
+  (junction (at 118.11 21.59) (diameter 0) (color 0 0 0 0)
   )
   (junction (at 281.94 86.36) (diameter 0) (color 0 0 0 0)
@@
     (stroke (width 0) (type default))
   )
+  (wire (pts (xy 138.43 21.59) (xy 144.145 21.59))
+    (stroke (width 0) (type default))
+  )
   (wire (pts (xy 30.48 157.48) (xy 34.925 157.48))
     (stroke (width 0) (type default))
@@
     (stroke (width 0) (type default))
   )
+  (wire (pts (xy 149.225 21.59) (xy 151.13 21.59))
+    (stroke (width 0) (type default))
+  )
   (wire (pts (xy 118.11 21.59) (xy 118.11 26.67))
     (stroke (width 0) (type default))
@@
   )
   (wire (pts (xy 166.37 151.765) (xy 169.545 151.765))
+    (stroke (width 0) (type default))
+  )
+  (wire (pts (xy 118.11 21.59) (xy 133.35 21.59))
     (stroke (width 0) (type default))
   )
@@
     (pin "2")
   )
+  (symbol (lib_id "Device:LED_Small") (at 146.685 21.59 180) (unit 1)
+    (in_bom yes) (on_board yes)
+    (default_instance (reference "U") (unit 1) (value "") (footprint ""))
+    (property "Reference" "U" (id 0) (at 146.685 16.51 0)
+      (effects (font (size 1.27 1.27)))
+    )
+    (property "Value" "" (id 1) (at 146.685 19.05 0)
+      (effects (font (size 1.27 1.27)))
+    )
+    (property "Footprint" "" (id 2) (at 146.685 21.59 90)
+      (effects (font (size 1.27 1.27)) hide)
+    )
+    (property "Datasheet" "~" (id 3) (at 146.685 21.59 90)
+      (effects (font (size 1.27 1.27)) hide)
+    )
+    (property "MPN" "150080VS75000" (id 4) (at 146.685 21.59 0)
+      (effects (font (size 1.27 1.27)) hide)
+    )
+    (pin "1")
+    (pin "2")
+  )
   (symbol (lib_id "Device:L_Ferrite_Coupled_1423") (at 81.28 37.465 0) (mirror x) (unit 1)
     (in_bom yes) (on_board yes) (fields_autoplaced)
@@
     )
     (property "MPN" "" (id 4) (at 125.095 155.575 0)
+      (effects (font (size 1.27 1.27)) hide)
+    )
+    (pin "1")
+    (pin "2")
+  )
+  (symbol (lib_id "Device:R_Small") (at 135.89 21.59 270) (mirror x) (unit 1)
+    (in_bom yes) (on_board yes)
+    (default_instance (reference "U") (unit 1) (value "") (footprint ""))
+    (property "Reference" "U" (id 0) (at 135.89 16.51 90)
+      (effects (font (size 1.27 1.27)))
+    )
+    (property "Value" "" (id 1) (at 135.89 19.05 90)
+      (effects (font (size 1.27 1.27)))
+    )
+    (property "Footprint" "" (id 2) (at 135.89 21.59 0)
+      (effects (font (size 1.27 1.27)) hide)
+    )
+    (property "Datasheet" "~" (id 3) (at 135.89 21.59 0)
+      (effects (font (size 1.27 1.27)) hide)
+    )
+    (property "MPN" "" (id 4) (at 135.89 21.59 90)
       (effects (font (size 1.27 1.27)) hide)
     )
@@
       (effects (font (size 1.27 1.27)) hide)
     )
+    (pin "1")
+  )
+  (symbol (lib_id "power:GND") (at 151.13 21.59 0) (unit 1)
+    (in_bom yes) (on_board yes)
+    (default_instance (reference "#PWR") (unit 1) (value "GND") (footprint ""))
+    (property "Reference" "#PWR" (id 0) (at 151.13 27.94 0)
+      (effects (font (size 1.27 1.27)) hide)
+    )
+    (property "Value" "GND" (id 1) (at 151.13 26.035 0)
+      (effects (font (size 1.27 1.27)))
+    )
+    (property "Footprint" "" (id 2) (at 151.13 21.59 0)
+      (effects (font (size 1.27 1.27)) hide)
+    )
+    (property "Datasheet" "" (id 3) (at 151.13 21.59 0)
+      (effects (font (size 1.27 1.27)) hide)
+    )

Commit message: hw: start working on rev4 controller
- removed SPI for display, and the associated SPI mux nonsense, and any
  superfluous resistors for pull-ups

- removed MAC address EEPROM

- start adding i2c RTC (which will also contain EEPROM with the MAC of
  the system, lol)

- start moving some components from bottom to top side of board

- tweaked positions of some mains voltage traces

- increased values of power indicator LED's current dropping resistors

- take 3V3 from SoM rather than generate it ourselves
Parts:
- added U: (no value), symbol Connector:TestPoint
Connections:
- net TRIGGER: now also U.1
Other:
- title: (none) -> Programmable Load Controller
Changed lines of the file:
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@@
 (kicad_sch (version 20220404) (generator eeschema)
   (paper "A4")
+  (title_block
+    (title "Programmable Load Controller")
+    (date "2022-06-28")
+    (rev "4")
+  )
   (junction (at 142.24 161.925) (diameter 0) (color 0 0 0 0)
   )
@@
   )
   (junction (at 100.33 146.685) (diameter 0) (color 0 0 0 0)
+  )
+  (junction (at 173.355 151.765) (diameter 0) (color 0 0 0 0)
   )
   (junction (at 113.03 50.165) (diameter 0) (color 0 0 0 0)
@@
     (stroke (width 0) (type default))
   )
-  (wire (pts (xy 166.37 151.765) (xy 169.545 151.765))
+  (wire (pts (xy 166.37 151.765) (xy 173.355 151.765))
     (stroke (width 0) (type default))
   )
@@
   )
   (wire (pts (xy 268.605 129.54) (xy 270.51 129.54))
+    (stroke (width 0) (type default))
+  )
+  (wire (pts (xy 173.355 151.765) (xy 182.88 151.765))
     (stroke (width 0) (type default))
   )
@@
     (effects (font (size 1.27 1.27)) (justify right))
   )
-  (hierarchical_label "TRIGGER" (shape output) (at 169.545 151.765 0) (fields_autoplaced)
+  (hierarchical_label "TRIGGER" (shape output) (at 182.88 151.765 0) (fields_autoplaced)
     (effects (font (size 1.27 1.27)) (justify left))
   )
@@
       (effects (font (size 1.27 1.27)) hide)
     )
+    (pin "1")
+  )
+  (symbol (lib_id "Connector:TestPoint") (at 173.355 151.765 0) (mirror y) (unit 1)
+    (in_bom yes) (on_board yes)
+    (default_instance (reference "U") (unit 1) (value "") (footprint ""))
+    (property "Reference" "U" (id 0) (at 175.26 147.1929 0)
+      (effects (font (size 1.27 1.27)) (justify right))
+    )
+    (property "Value" "" (id 1) (at 175.26 149.7329 0)
+      (effects (font (size 1.27 1.27)) (justify right))
+    )
+    (property "Footprint" "" (id 2) (at 168.275 151.765 0)
+      (effects (font (size 1.27 1.27)) hide)
+    )
+    (property "Datasheet" "~" (id 3) (at 168.275 151.765 0)
+      (effects (font (size 1.27 1.27)) hide)
+    )
+    (property "Color" "Yellow" (id 4) (at 173.355 151.765 0)
+      (effects (font (size 1.27 1.27)) hide)
+    )
+    (property "MPN" "5004" (id 5) (at 173.355 151.765 0)
+      (effects (font (size 1.27 1.27)) hide)
+    )

Commit message: hw: revise USB power stuff
- fixed the remaining usb powering stuff for the front panel host
  connector

- replaced 33µF SMD caps with through-hole equivalents

- removed some of the bottom mounted components for analog board power
  connection
Parts:
- U: MPN A768EB336M1GLAE045 -> A758EK226M1EAAE050
Changed lines of the file:
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@@
-    (stroke (width 0) (type default))
-  )
-  (wire (pts (xy 66.04 95.885) (xy 81.28 95.885))
     (stroke (width 0) (type default))
   )
@@
   (hierarchical_label "ETH_TXP" (shape input) (at 245.11 76.2 180) (fields_autoplaced)
     (effects (font (size 1.27 1.27)) (justify right))
+  )
+  (symbol (lib_id "power:+12V") (at 81.28 95.885 0) (unit 1)
+    (in_bom yes) (on_board yes)
+    (default_instance (reference "U") (unit 1) (value "") (footprint ""))
+    (property "Reference" "U" (id 0) (at 81.28 99.695 0)
+      (effects (font (size 1.27 1.27)) hide)
+    )
+    (property "Value" "" (id 1) (at 81.28 91.44 0)
+      (effects (font (size 1.27 1.27)))
+    )
+    (property "Footprint" "" (id 2) (at 81.28 95.885 0)
+      (effects (font (size 1.27 1.27)) hide)
+    )
+    (property "Datasheet" "" (id 3) (at 81.28 95.885 0)
+      (effects (font (size 1.27 1.27)) hide)
+    )
+    (pin "1")
   )
   (symbol (lib_id "Device:C_Small") (at 160.02 171.45 0) (mirror x) (unit 1)
@@
       (effects (font (size 1.27 1.27)) hide)
     )
-    (property "MPN" "A768EB336M1GLAE045" (id 4) (at 81.28 98.425 0)
-      (effects (font (size 1.27 1.27)) hide)
-    )
+    (property "MPN" "A758EK226M1EAAE050" (id 4) (at 81.28 98.425 0)
+      (effects (font (size 1.27 1.27)) hide)
+    )

Commit message: hw: finish power section rework
- Changed the +5V supply to also use a new discrete regulator

- Moved fan controller to where the VBus LED is, so that the connector
  is easily accessible even with the analog board mounted in its card
  guides
Parts:
- added C: C_Small, symbol Device:C_Small
Connections:
- net +12V: now also C.1
- net GND: now also C.2
Other:
- moved on the sheet: U
Changed lines of the file:
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@@
+    (stroke (width 0) (type default))
+  )
+  (wire (pts (xy 66.04 95.885) (xy 78.105 95.885))
     (stroke (width 0) (type default))
   )
@@
     (effects (font (size 1.27 1.27)) (justify right))
   )
-  (symbol (lib_id "power:+12V") (at 81.28 95.885 0) (unit 1)
-    (in_bom yes) (on_board yes)
-    (default_instance (reference "U") (unit 1) (value "") (footprint ""))
-    (property "Reference" "U" (id 0) (at 81.28 99.695 0)
-      (effects (font (size 1.27 1.27)) hide)
-    )
-    (property "Value" "" (id 1) (at 81.28 91.44 0)
-      (effects (font (size 1.27 1.27)))
-    )
-    (property "Footprint" "" (id 2) (at 81.28 95.885 0)
-      (effects (font (size 1.27 1.27)) hide)
-    )
-    (property "Datasheet" "" (id 3) (at 81.28 95.885 0)
+  (symbol (lib_id "power:+12V") (at 145.415 31.75 0) (unit 1)
+    (in_bom yes) (on_board yes)
+    (default_instance (reference "U") (unit 1) (value "") (footprint ""))
+    (property "Reference" "U" (id 0) (at 145.415 35.56 0)
+      (effects (font (size 1.27 1.27)) hide)
+    )
+    (property "Value" "" (id 1) (at 145.415 27.305 0)
+      (effects (font (size 1.27 1.27)))
+    )
+    (property "Footprint" "" (id 2) (at 145.415 31.75 0)
+      (effects (font (size 1.27 1.27)) hide)
+    )
+    (property "Datasheet" "" (id 3) (at 145.415 31.75 0)
       (effects (font (size 1.27 1.27)) hide)
     )
@@
     (pin "6")
   )
-  (symbol (lib_id "Device:C_Polarized_Small") (at 81.28 98.425 0) (unit 1)
-    (in_bom yes) (on_board yes)
-    (default_instance (reference "U") (unit 1) (value "") (footprint ""))
-    (property "Reference" "U" (id 0) (at 83.82 98.425 0)
+  (symbol (lib_id "Device:C_Polarized_Small") (at 145.415 34.29 0) (unit 1)
+    (in_bom yes) (on_board yes)
+    (default_instance (reference "U") (unit 1) (value "") (footprint ""))
+    (property "Reference" "U" (id 0) (at 147.955 34.29 0)
       (effects (font (size 1.27 1.27)) (justify left))
     )
-    (property "Value" "" (id 1) (at 83.82 100.965 0)
+    (property "Value" "" (id 1) (at 147.955 36.83 0)
       (effects (font (size 1.27 1.27)) (justify left))
     )
-    (property "Footprint" "" (id 2) (at 81.28 98.425 0)
-      (effects (font (size 1.27 1.27)) hide)
-    )
-    (property "Datasheet" "~" (id 3) (at 81.28 98.425 0)
-      (effects (font (size 1.27 1.27)) hide)
-    )
-    (property "MPN" "A758EK226M1EAAE050" (id 4) (at 81.28 98.425 0)
+    (property "Footprint" "" (id 2) (at 145.415 34.29 0)
+      (effects (font (size 1.27 1.27)) hide)
+    )
+    (property "Datasheet" "~" (id 3) (at 145.415 34.29 0)
+      (effects (font (size 1.27 1.27)) hide)
+    )
+    (property "MPN" "A758EK226M1EAAE050" (id 4) (at 145.415 34.29 0)
       (effects (font (size 1.27 1.27)) hide)
     )
@@
     (pin "2")
   )
+  (symbol (lib_id "Device:C_Small") (at 78.105 98.425 0) (unit 1)
+    (in_bom yes) (on_board yes)
+    (default_instance (reference "C") (unit 1) (value "C_Small") (footprint ""))
+    (property "Reference" "C" (id 0) (at 80.645 97.155 0)
+      (effects (font (size 1.27 1.27)) (justify left))
+    )
+    (property "Value" "C_Small" (id 1) (at 80.645 99.695 0)
+      (effects (font (size 1.27 1.27)) (justify left))
+    )
+    (property "Footprint" "" (id 2) (at 78.105 98.425 0)
+      (effects (font (size 1.27 1.27)) hide)
+    )
+    (property "Datasheet" "~" (id 3) (at 78.105 98.425 0)
+      (effects (font (size 1.27 1.27)) hide)
+    )
+    (property "JLPCB" "C15850" (id 4) (at 78.105 98.425 0)
+      (effects (font (size 1.27 1.27)) hide)
+    )
+    (pin "1")
+    (pin "2")
+  )
   (symbol (lib_id "Isolator:FODM217B") (at 111.76 149.225 0) (unit 1)
     (in_bom yes) (on_board yes) (fields_autoplaced)
@@
     (pin "1")
   )
-  (symbol (lib_id "power:GND") (at 81.28 100.965 0) (unit 1)
-    (in_bom yes) (on_board yes) (fields_autoplaced)
-    (default_instance (reference "U") (unit 1) (value "") (footprint ""))
-    (property "Reference" "U" (id 0) (at 81.28 107.315 0)
-      (effects (font (size 1.27 1.27)) hide)
-    )
-    (property "Value" "" (id 1) (at 81.28 105.41 0)
-      (effects (font (size 1.27 1.27)))
-    )
-    (property "Footprint" "" (id 2) (at 81.28 100.965 0)
-      (effects (font (size 1.27 1.27)) hide)
-    )
-    (property "Datasheet" "" (id 3) (at 81.28 100.965 0)
+  (symbol (lib_id "power:GND") (at 145.415 36.83 0) (unit 1)
+    (in_bom yes) (on_board yes) (fields_autoplaced)
+    (default_instance (reference "U") (unit 1) (value "") (footprint ""))
+    (property "Reference" "U" (id 0) (at 145.415 43.18 0)
+      (effects (font (size 1.27 1.27)) hide)
+    )
+    (property "Value" "" (id 1) (at 145.415 41.275 0)
+      (effects (font (size 1.27 1.27)))
+    )
+    (property "Footprint" "" (id 2) (at 145.415 36.83 0)
+      (effects (font (size 1.27 1.27)) hide)
+    )
+    (property "Datasheet" "" (id 3) (at 145.415 36.83 0)
       (effects (font (size 1.27 1.27)) hide)
     )
@@
     (pin "2")
   )
+  (symbol (lib_id "power:GND") (at 78.105 100.965 0) (unit 1)
+    (in_bom yes) (on_board yes) (fields_autoplaced)
+    (default_instance (reference "#PWR") (unit 1) (value "GND") (footprint ""))
+    (property "Reference" "#PWR" (id 0) (at 78.105 107.315 0)
+      (effects (font (size 1.27 1.27)) hide)
+    )
+    (property "Value" "GND" (id 1) (at 78.105 105.41 0)
+      (effects (font (size 1.27 1.27)))
+    )
+    (property "Footprint" "" (id 2) (at 78.105 100.965 0)
+      (effects (font (size 1.27 1.27)) hide)
+    )
+    (property "Datasheet" "" (id 3) (at 78.105 100.965 0)
+      (effects (font (size 1.27 1.27)) hide)
+    )
+    (pin "1")
+  )
   (symbol (lib_id "power:GND") (at 30.48 162.56 0) (unit 1)

Commit message: hw: add charger for RTC
- added RTC supercapacitor

- added the charging circuit for the RTC (with adjustment for voltage
  and all that fun stuff) based around a bonus linear regulator for the
  supercap

- minor tweaks all around: add more JLCPCB part numbers and fixed some
  footprints for some components
Parts:
- U: JLCPCB (none) -> C25804
Changed lines of the file:
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@@
+      (effects (font (size 1.27 1.27)) hide)
+    )
+    (property "JLCPCB" "C25804" (id 4) (at 39.37 98.425 0)
       (effects (font (size 1.27 1.27)) hide)
     )

Commit message: hw: add more jlcpcb p/n; minor cleanup
- added jlcpcb part numbers for various resistors and passives

- minor clean up of stuff on the board, including moving the +VDC
  indicator LED and widening the fastener slot for the RTC supercap
Parts:
- removed U: (no value), symbol Diode:SM4007
- added D: SM4007, Diode_SMD:D_MELF, symbol Diode:SM4007
- U: JLCPCB (none) -> C23138
- U: JLCPCB (none) -> C23162
- U: JLCPCB (none) -> C23234
- U: JLCPCB (none) -> C25804
Connections:
- net +12V: now also D.1 (K)
- net at K.12, U.3 (C): now also D.2 (A)
Changed lines of the file:
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@@
+    (pin "2")
+  )
+  (symbol (lib_id "Diode:SM4007") (at 85.725 45.085 0) (unit 1)
+    (in_bom yes) (on_board yes)
+    (default_instance (reference "D") (unit 1) (value "SM4007") (footprint "Diode_SMD:D_MELF"))
+    (property "Reference" "D" (id 0) (at 85.725 49.53 0)
+      (effects (font (size 1.27 1.27)))
+    )
+    (property "Value" "SM4007" (id 1) (at 85.725 52.07 0)
+      (effects (font (size 1.27 1.27)))
+    )
+    (property "Footprint" "Diode_SMD:D_MELF" (id 2) (at 85.725 49.53 0)
+      (effects (font (size 1.27 1.27)) hide)
+    )
+    (property "Datasheet" "http://cdn-reichelt.de/documents/datenblatt/A400/SMD1N400%23DIO.pdf" (id 3) (at 85.725 45.085 0)
+      (effects (font (size 1.27 1.27)) hide)
+    )
+    (property "MPN" "FM4007W-W" (id 4) (at 85.725 45.085 0)
+      (effects (font (size 1.27 1.27)) hide)
+    )
+    (pin "1")
     (pin "2")
   )
@@
     )
     (property "MPN" "" (id 4) (at 240.665 88.9 90)
+      (effects (font (size 1.27 1.27)) hide)
+    )
+    (property "JLCPCB" "C23138" (id 5) (at 240.665 88.9 90)
       (effects (font (size 1.27 1.27)) hide)
     )
@@
     )
     (property "MPN" "" (id 4) (at 220.98 91.44 90)
+      (effects (font (size 1.27 1.27)) hide)
+    )
+    (property "JLCPCB" "C23138" (id 5) (at 220.98 91.44 0)
       (effects (font (size 1.27 1.27)) hide)
     )
@@
       (effects (font (size 1.27 1.27)) hide)
     )
+    (property "JLCPCB" "C23162" (id 4) (at 58.42 98.425 0)
+      (effects (font (size 1.27 1.27)) hide)
+    )
     (pin "1")
     (pin "2")
@@
       (effects (font (size 1.27 1.27)) hide)
     )
+    (property "JLCPCB" "C23234" (id 5) (at 135.89 21.59 90)
+      (effects (font (size 1.27 1.27)) hide)
+    )
     (pin "1")
     (pin "2")
@@
     (pin "2")
     (pin "3")
-  )
-  (symbol (lib_id "Diode:SM4007") (at 85.725 45.085 0) (unit 1)
-    (in_bom yes) (on_board yes)
-    (default_instance (reference "U") (unit 1) (value "") (footprint ""))
-    (property "Reference" "U" (id 0) (at 85.725 52.07 0)
-      (effects (font (size 1.27 1.27)))
-    )
-    (property "Value" "" (id 1) (at 85.725 49.53 0)
-      (effects (font (size 1.27 1.27)))
-    )
-    (property "Footprint" "" (id 2) (at 85.725 49.53 0)
-      (effects (font (size 1.27 1.27)) hide)
-    )
-    (property "Datasheet" "http://cdn-reichelt.de/documents/datenblatt/A400/SMD1N400%23DIO.pdf" (id 3) (at 85.725 45.085 0)
-      (effects (font (size 1.27 1.27)) hide)
-    )
-    (property "MPN" "FM4007W-W" (id 4) (at 85.725 45.085 0)
-      (effects (font (size 1.27 1.27)) hide)
-    )
-    (pin "1")
-    (pin "2")
   )
   (symbol (lib_id "programmable-load:EMC2101-R") (at 43.815 147.32 0) (unit 1)
@@
       (effects (font (size 1.27 1.27)) hide)
     )
+    (property "JLCPCB" "C25804" (id 4) (at 45.72 184.15 90)
+      (effects (font (size 1.27 1.27)) hide)
+    )
