File: Hardware/controller/analog-io.kicad_sch (KiCad schematic)
At the start: 8 parts

Commit message: replace 22µF caps with 47µF
- these are a bit cheaper and give us more capacitance, hell yeah
  brother
Parts:
- U: MPN A758EK226M1EAAE050 -> A750EK476M1EAAE040
Changed lines of the file:
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@@
       (effects (font (size 1.27 1.27)) hide)
     )
-    (property "MPN" "A758EK226M1EAAE050" (id 4) (at 91.44 40.005 0)
+    (property "MPN" "A750EK476M1EAAE040" (id 4) (at 91.44 40.005 0)
       (effects (font (size 1.27 1.27)) hide)
     )

Commit message: added touch controller reset/irq lines
Parts:
- U: MPN 0ZCJ0050FF2G -> 0ZCJ0050AF2E
Changed lines of the file:
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@@
       (effects (font (size 1.27 1.27)) hide)
     )
-    (property "MPN" "0ZCJ0050FF2G" (id 4) (at 33.02 33.655 90)
+    (property "MPN" "0ZCJ0050AF2E" (id 4) (at 33.02 33.655 90)
       (effects (font (size 1.27 1.27)) hide)
     )
