File: Hardware/controller/rtc.kicad_sch (KiCad schematic)
At the start: 17 parts

Commit message: hw: fix part numbers
- fixed missing or incorrect MPN and JLCPCB part numbers for various
  components; most should have either one of these now
Parts:
- C: JLCPCB (none) -> C15850; JLPCB C15850 -> (none)
- U: MPN (none) -> MCP79410T-I/ST
- U: MPN (none) -> AP2202K-ADJTRG1
Changed lines of the file:
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@@
       (effects (font (size 1.27 1.27)) hide)
     )
-    (property "JLPCB" "C15850" (id 4) (at 116.84 88.265 0)
+    (property "JLCPCB" "C15850" (id 4) (at 116.84 88.265 0)
       (effects (font (size 1.27 1.27)) hide)
     )
@@
     )
     (property "Datasheet" "https://ww1.microchip.com/downloads/en/DeviceDoc/MCP79410-MCP79411-MCP79412-Battery-Backed%20I2C-RTCC-20002266J.pdf" (id 3) (at 40.64 15.875 0)
+      (effects (font (size 1.27 1.27)) hide)
+    )
+    (property "MPN" "MCP79410T-I/ST" (id 4) (at 39.37 39.37 0)
       (effects (font (size 1.27 1.27)) hide)
     )
@@
       (effects (font (size 1.27 1.27)) hide)
     )
+    (property "MPN" "AP2202K-ADJTRG1" (id 4) (at 88.9 83.82 0)
+      (effects (font (size 1.27 1.27)) hide)
+    )

Commit message: Minor tweaks to controller board
- Removed I2C mux: use I2C6 as a separate bus for the on-board stuff

- Replaced RTC with MCP79401 in MSOP package

- Tweaks to fan controller circuit

- Embiggened board around IO connectors, and moved the connectors .5mm
  further out so they make better contact with the panels

- Replace trimpots with cheaper versions

- Other relatively minor tweaks to the locations of ext trigger/aux out
  signal conditioning circuitry

- Moved the +12V fuse for analog board so it's not as precariously next
  to the front panel connector
Parts:
- RV: MPN 3296Y-1-103LF -> CT-94EY103
- U: MPN MCP79410T-I/ST -> MCP79401-I/MS
Changed lines of the file:
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@@
       (effects (font (size 1.27 1.27)) hide)
     )
-    (property "MPN" "3296Y-1-103LF" (id 4) (at 105.41 100.965 0)
+    (property "MPN" "CT-94EY103" (id 4) (at 105.41 100.965 0)
       (effects (font (size 1.27 1.27)) hide)
     )
@@
       (effects (font (size 1.27 1.27)) hide)
     )
-    (property "MPN" "MCP79410T-I/ST" (id 4) (at 39.37 39.37 0)
+    (property "MPN" "MCP79401-I/MS" (id 4) (at 39.37 39.37 0)
       (effects (font (size 1.27 1.27)) hide)
     )
