File: Hardware/front/display.kicad_sch (KiCad schematic)
At the start: 7 parts

Commit message: Start routing front panel stuff
- Routed some of the LED driver pins and replaced footprints of passives
  with 0603 size to match the controller board
Parts:
- U: MPN CL21B104KACNFNC -> (none)
Changed lines of the file:
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@@
       (effects (font (size 1.27 1.27)) hide)
     )
-    (property "MPN" "CL21B104KACNFNC" (id 4) (at 257.175 49.53 0)
+    (property "MPN" "" (id 4) (at 257.175 49.53 0)
       (effects (font (size 1.27 1.27)) hide)
     )

Commit message: Finished routing front panel
- Finished routing the contents of the front panel; it could probably
  use an optimization pass and general cleanup.

  A few of the assignments of IOs/LED driver outputs were changed as
  well to make the routing less of a pain in the ass, as compared to the
  previous front panels.

- Minor tweaks to controller to remove some unused signals
Parts:
- added R: R_Small, symbol Device:R_Small
Connections:
- net +3V3: now also R.1
- net ~{TOUCH_IRQ}: now also R.2
Changed lines of the file:
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@@
+    (stroke (width 0) (type default))
+  )
+  (wire (pts (xy 205.74 146.05) (xy 215.9 146.05))
     (stroke (width 0) (type default))
   )
@@
     (effects (font (size 1.27 1.27)) (justify left bottom))
   )
+  (label "~{TOUCH_IRQ}" (at 215.9 146.05 0) (fields_autoplaced)
+    (effects (font (size 1.27 1.27)) (justify right bottom))
+  )
   (label "R2" (at 217.17 72.39 0) (fields_autoplaced)
     (effects (font (size 1.27 1.27)) (justify right bottom))
@@
   (hierarchical_label "SPI_MOSI" (shape input) (at 231.14 59.69 0) (fields_autoplaced)
     (effects (font (size 1.27 1.27)) (justify left))
+  )
+  (symbol (lib_id "Device:R_Small") (at 203.2 146.05 90) (unit 1)
+    (in_bom yes) (on_board yes) (fields_autoplaced)
+    (default_instance (reference "R") (unit 1) (value "R_Small") (footprint ""))
+    (property "Reference" "R" (id 0) (at 203.2 140.97 90)
+      (effects (font (size 1.27 1.27)))
+    )
+    (property "Value" "R_Small" (id 1) (at 203.2 143.51 90)
+      (effects (font (size 1.27 1.27)))
+    )
+    (property "Footprint" "" (id 2) (at 203.2 146.05 0)
+      (effects (font (size 1.27 1.27)) hide)
+    )
+    (property "Datasheet" "~" (id 3) (at 203.2 146.05 0)
+      (effects (font (size 1.27 1.27)) hide)
+    )
+    (pin "1")
+    (pin "2")
   )
   (symbol (lib_id "Device:C_Small") (at 257.175 49.53 0) (unit 1)
@@
       (effects (font (size 1.27 1.27)) hide)
     )
+    (pin "1")
+  )
+  (symbol (lib_id "power:+3V3") (at 200.66 146.05 90) (unit 1)
+    (in_bom yes) (on_board yes)
+    (default_instance (reference "#PWR") (unit 1) (value "+3V3") (footprint ""))
+    (property "Reference" "#PWR" (id 0) (at 204.47 146.05 0)
+      (effects (font (size 1.27 1.27)) hide)
+    )
+    (property "Value" "+3V3" (id 1) (at 197.485 146.05 90)
+      (effects (font (size 1.27 1.27)) (justify left))
+    )
+    (property "Footprint" "" (id 2) (at 200.66 146.05 0)
+      (effects (font (size 1.27 1.27)) hide)
+    )
+    (property "Datasheet" "" (id 3) (at 200.66 146.05 0)
+      (effects (font (size 1.27 1.27)) hide)
+    )

Commit message: Minor tweaks to front panel & controller for manufacture
- Create footprint for JLCPCB assembly tooling holes

- Added tooling holes to front panel board and fixed ERC errors

- Added tooling holes to controller

- Moved a few traces on controller board and fixed a few broken package
  associations

- Add pull-up on Ethernet PHY's reset line (so when the SoM boots, we're
  not making it angerey)

- Fixed order of BOOTx pins to DIP switch

- Fixed swapped USB host/device pins

- Fixed swapped ETH_TXP/ETH_TXN pair on when exiting the CPU sheet and
  connecting to the rear IO sheet (in the main sheet of the schematic)
  and the associated incorrect resistors/caps
Parts:
- added R: R_Small, symbol Device:R_Small
Connections:
- net +3V3: now also R.2
- net BACKLIGHT: now also R.1
Other:
- note added: "Ensure backlight is off when undriven"
Changed lines of the file:
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@@
+    (stroke (width 0) (type default))
+  )
+  (wire (pts (xy 53.34 76.2) (xy 54.61 76.2))
     (stroke (width 0) (type default))
   )
@@
   )
   (text "Set RGB + SPI (SCK rising trigger)" (at 241.3 115.57 0)
+    (effects (font (size 1.27 1.27)) (justify left bottom))
+  )
+  (text "Ensure backlight is off when undriven" (at 38.1 69.215 0)
     (effects (font (size 1.27 1.27)) (justify left bottom))
   )
@@
   )
   (hierarchical_label "~{TOUCH_IRQ}" (shape output) (at 231.14 34.29 0) (fields_autoplaced)
+    (effects (font (size 1.27 1.27)) (justify left))
+  )
+  (hierarchical_label "BACKLIGHT" (shape input) (at 54.61 76.2 0) (fields_autoplaced)
     (effects (font (size 1.27 1.27)) (justify left))
   )
@@
     (pin "1")
   )
+  (symbol (lib_id "power:+3V3") (at 48.26 76.2 90) (unit 1)
+    (in_bom yes) (on_board yes)
+    (default_instance (reference "#PWR") (unit 1) (value "+3V3") (footprint ""))
+    (property "Reference" "#PWR" (id 0) (at 52.07 76.2 0)
+      (effects (font (size 1.27 1.27)) hide)
+    )
+    (property "Value" "+3V3" (id 1) (at 45.085 76.2 90)
+      (effects (font (size 1.27 1.27)) (justify left))
+    )
+    (property "Footprint" "" (id 2) (at 48.26 76.2 0)
+      (effects (font (size 1.27 1.27)) hide)
+    )
+    (property "Datasheet" "" (id 3) (at 48.26 76.2 0)
+      (effects (font (size 1.27 1.27)) hide)
+    )
+    (pin "1")
+  )
   (symbol (lib_id "power:GND") (at 67.945 55.245 0) (unit 1)
     (in_bom yes) (on_board yes)
@@
     (pin "1")
   )
+  (symbol (lib_id "Device:R_Small") (at 50.8 76.2 270) (unit 1)
+    (in_bom yes) (on_board yes) (fields_autoplaced)
+    (default_instance (reference "R") (unit 1) (value "R_Small") (footprint ""))
+    (property "Reference" "R" (id 0) (at 50.8 71.12 90)
+      (effects (font (size 1.27 1.27)))
+    )
+    (property "Value" "R_Small" (id 1) (at 50.8 73.66 90)
+      (effects (font (size 1.27 1.27)))
+    )
+    (property "Footprint" "" (id 2) (at 50.8 76.2 0)
+      (effects (font (size 1.27 1.27)) hide)
+    )
+    (property "Datasheet" "~" (id 3) (at 50.8 76.2 0)
+      (effects (font (size 1.27 1.27)) hide)
+    )
+    (pin "1")
+    (pin "2")
+  )
   (symbol (lib_id "power:GND") (at 267.97 52.07 0) (unit 1)

Commit message: hw: start work on new front panel board
- This replaces all the various I2C chips with a single RP2040 (with
  some boot flash) to handle scanning the keyboard, driving PWM LEDs
  (including the display backlight) and actually handling the display
  controller initialization.

- Flipped the pinout of the connector to the main controller board
Parts:
- added U: (no value), symbol Device:R_Small
Connections:
- net +3V3: now also U.2
- net ~{SPI_CS}: now also U.1
Changed lines of the file:
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@@
   (title_block
     (title "Front Panel")
-    (date "2022-05-20")
-    (rev "2")
+    (date "2022-06-27")
+    (rev "4")
   )
   (junction (at 229.87 46.99) (diameter 0) (color 0 0 0 0)
@@
   (junction (at 266.7 122.555) (diameter 0) (color 0 0 0 0)
   )
+  (junction (at 48.26 76.2) (diameter 0) (color 0 0 0 0)
+  )
   (junction (at 266.7 141.605) (diameter 0) (color 0 0 0 0)
   )
@@
     (stroke (width 0) (type default))
   )
+  (wire (pts (xy 48.26 76.2) (xy 48.26 85.09))
+    (stroke (width 0) (type default))
+  )
   (wire (pts (xy 229.87 52.07) (xy 242.57 52.07))
     (stroke (width 0) (type default))
@@
   )
   (wire (pts (xy 215.9 57.15) (xy 217.17 57.15))
+    (stroke (width 0) (type default))
+  )
+  (wire (pts (xy 53.34 85.09) (xy 54.61 85.09))
     (stroke (width 0) (type default))
   )
@@
   )
   (hierarchical_label "SPI_MOSI" (shape input) (at 231.14 59.69 0) (fields_autoplaced)
+    (effects (font (size 1.27 1.27)) (justify left))
+  )
+  (hierarchical_label "~{SPI_CS}" (shape input) (at 54.61 85.09 0) (fields_autoplaced)
     (effects (font (size 1.27 1.27)) (justify left))
   )
@@
     (pin "1")
   )
+  (symbol (lib_id "Device:R_Small") (at 50.8 85.09 270) (mirror x) (unit 1)
+    (in_bom yes) (on_board yes)
+    (default_instance (reference "U") (unit 1) (value "") (footprint ""))
+    (property "Reference" "U" (id 0) (at 50.8 80.01 90)
+      (effects (font (size 1.27 1.27)))
+    )
+    (property "Value" "" (id 1) (at 50.8 82.55 90)
+      (effects (font (size 1.27 1.27)))
+    )
+    (property "Footprint" "" (id 2) (at 50.8 85.09 0)
+      (effects (font (size 1.27 1.27)) hide)
+    )
+    (property "Datasheet" "~" (id 3) (at 50.8 85.09 0)
+      (effects (font (size 1.27 1.27)) hide)
+    )
+    (property "MPN" "" (id 4) (at 50.8 85.09 90)
+      (effects (font (size 1.27 1.27)) hide)
+    )
+    (pin "1")
+    (pin "2")
+  )
   (symbol (lib_id "Device:R_Small") (at 39.37 40.64 0) (unit 1)

Commit message: hw: more front panel stuff
- fixed the mirrored pinout for the connector to the controller board

- Replaced a few capacitors to reduce BOM count

- Start connecting signals to RP2040, including the flash connection
  (dedicated to it)
Parts:
- removed C: C_Polarized_Small, symbol Device:C_Polarized_Small
- removed Q (x2): 2N7002E, Package_TO_SOT_SMD:SOT-23, symbol Transistor_FET:2N7002H
- removed R (x2): R_Small, symbol Device:R_Small
- added Q: AO3400A, Package_TO_SOT_SMD:SOT-23, symbol Transistor_FET:AO3400A
- added R: R_Small, symbol Device:R_Small
- added U: (no value), symbol Device:C_Small
- J: symbol Connector_Generic_MountingPin:Conn_02x25_Counter_Clockwise_MountingPin -> Connector_Generic:Conn_02x25_Counter_Clockwise
Connections:
- net LEDK2 is gone; now on net LEDK: J.3 (Pin_3)
- net +3V3: now also U.1
- net BACKLIGHT: now also Q.1 (G)
- net GND: now also Q.2 (S), U.2; no longer J.MP (MountPin)
- net LEDK1 renamed LEDK
- net LEDK: now also R.1
- new net: Q.3 (D), R.2
