File: Hardware/front/display.kicad_sch (KiCad schematic)
At the start: 9 parts

Commit message: Rev4 front panel (#3)
* hw: start work on new front panel board

- This replaces all the various I2C chips with a single RP2040 (with
  some boot flash) to handle scanning the keyboard, driving PWM LEDs
  (including the display backlight) and actually handling the display
  controller initialization.

- Flipped the pinout of the connector to the main controller board

* hw: more front panel stuff

- fixed the mirrored pinout for the connector to the controller board

- Replaced a few capacitors to reduce BOM count

- Start connecting signals to RP2040, including the flash connection
  (dedicated to it)

* hw: First pass at new front panel

- Finished routing all signals on the front panel

- Put back the LED controller (PCA9955B) since that's a very nice and
  convenient way to drive the LEDs; it's driven via a "private" I2C bus
  from the RP2040 instead of the host controlling it.

  The touch panel controller is also hanging off this private bus so we
  can deal with it.

- Made trigger LED bicolor (green/orange)

* hw: minor front panel tweaks

* updated front panel pinout

- added system reset, direct load on/off switch output lines

- added separate touch screen reset/interrupt lines (the touch
  controller gets to be driven by linux side)

- update footprint for ER-TFT040-1 display

  this tweaks the sizes of the openings and the text labels a bit to be
  prettier

* swap touch irq/reset lines to match controller
Parts:
- removed C: C_Polarized_Small, symbol Device:C_Polarized_Small
- removed Q (x2): 2N7002E, Package_TO_SOT_SMD:SOT-23, symbol Transistor_FET:2N7002H
- removed R (x3): R_Small, symbol Device:R_Small
- added N: Housing, symbol Mechanical:Housing
- added Q: AO3400A, Package_TO_SOT_SMD:SOT-23, symbol Transistor_FET:AO3400A
- added R: R_Small, symbol Device:R_Small
- added TP (x4): TestPoint, symbol Connector:TestPoint
- added U (x2): (no value), symbol Device:R_Small
- added U: (no value), symbol Device:C_Small
- J: symbol Connector_Generic_MountingPin:Conn_02x25_Counter_Clockwise_MountingPin -> Connector_Generic:Conn_02x25_Counter_Clockwise; JLCPCB (none) -> C231436
- R: JLCPCB (none) -> C25804
- U: JLCPCB (none) -> C14663
Connections:
- net LEDK2 is gone; now on net LEDK: J.3 (Pin_3)
- net +3V3: now also U.1, U.2, U.2; no longer R.2
- net BACKLIGHT: now also Q.1 (G)
- net GND: now also R.2, Q.2 (S), U.2; no longer J.MP (MountPin)
- net SPI_MISO: now also TP.1
- net SPI_MOSI: now also TP.1
- net SPI_SCK: now also TP.1
- net ~{SPI_CS}: now also TP.1, U.1
- net ~{TOUCH_RESET}: now also U.1
- net LEDK1 renamed LEDK
- net LEDK: now also R.1
- new net: Q.3 (D), R.2
