File: Hardware/front/buttons.kicad_sch (KiCad schematic)
At the start: 40 parts

Commit message: Rev4 front panel (#3)
* hw: start work on new front panel board

- This replaces all the various I2C chips with a single RP2040 (with
  some boot flash) to handle scanning the keyboard, driving PWM LEDs
  (including the display backlight) and actually handling the display
  controller initialization.

- Flipped the pinout of the connector to the main controller board

* hw: more front panel stuff

- fixed the mirrored pinout for the connector to the controller board

- Replaced a few capacitors to reduce BOM count

- Start connecting signals to RP2040, including the flash connection
  (dedicated to it)

* hw: First pass at new front panel

- Finished routing all signals on the front panel

- Put back the LED controller (PCA9955B) since that's a very nice and
  convenient way to drive the LEDs; it's driven via a "private" I2C bus
  from the RP2040 instead of the host controlling it.

  The touch panel controller is also hanging off this private bus so we
  can deal with it.

- Made trigger LED bicolor (green/orange)

* hw: minor front panel tweaks

* updated front panel pinout

- added system reset, direct load on/off switch output lines

- added separate touch screen reset/interrupt lines (the touch
  controller gets to be driven by linux side)

- update footprint for ER-TFT040-1 display

  this tweaks the sizes of the openings and the text labels a bit to be
  prettier

* swap touch irq/reset lines to match controller
Parts:
- R, U: JLCPCB (none) -> C25804
- U: JLCPCB (none) -> C21190
- U: JLCPCB (none) -> C19666
- U: JLCPCB (none) -> C14663
Changed lines of the file:
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@@
   (title_block
     (title "Front Panel")
-    (date "2022-05-20")
-    (rev "2")
+    (date "2022-06-27")
+    (rev "4")
   )
   (junction (at 61.595 73.025) (diameter 0) (color 0 0 0 0)
@@
       (effects (font (size 1.27 1.27)) hide)
     )
+    (property "JLCPCB" "C21190" (id 5) (at 33.655 31.115 0)
+      (effects (font (size 1.27 1.27)) hide)
+    )
     (pin "1")
     (pin "2")
@@
       (effects (font (size 1.27 1.27)) hide)
     )
+    (property "JLCPCB" "C21190" (id 5) (at 223.52 34.925 0)
+      (effects (font (size 1.27 1.27)) hide)
+    )
     (pin "1")
     (pin "2")
@@
     )
     (property "MPN" "" (id 4) (at 33.655 88.265 0)
+      (effects (font (size 1.27 1.27)) hide)
+    )
+    (property "JLCPCB" "C21190" (id 5) (at 33.655 88.265 0)
       (effects (font (size 1.27 1.27)) hide)
     )
@@
       (effects (font (size 1.27 1.27)) hide)
     )
+    (property "JLCPCB" "C21190" (id 5) (at 212.09 69.85 90)
+      (effects (font (size 1.27 1.27)) hide)
+    )
     (pin "1")
     (pin "2")
@@
       (effects (font (size 1.27 1.27)) hide)
     )
+    (property "JLCPCB" "C19666" (id 5) (at 61.595 85.09 0)
+      (effects (font (size 1.27 1.27)) hide)
+    )
     (pin "1")
     (pin "2")
@@
       (effects (font (size 1.27 1.27)) hide)
     )
+    (property "JLCPCB" "C25804" (id 5) (at 215.265 34.925 0)
+      (effects (font (size 1.27 1.27)) hide)
+    )
     (pin "1")
     (pin "2")
@@
       (effects (font (size 1.27 1.27)) hide)
     )
+    (property "JLCPCB" "C25804" (id 4) (at 217.805 46.99 90)
+      (effects (font (size 1.27 1.27)) hide)
+    )
     (pin "1")
     (pin "2")
@@
     )
     (property "MPN" "" (id 4) (at 25.4 69.215 0)
+      (effects (font (size 1.27 1.27)) hide)
+    )
+    (property "JLCPCB" "C25804" (id 5) (at 25.4 69.215 0)
       (effects (font (size 1.27 1.27)) hide)
     )
@@
       (effects (font (size 1.27 1.27)) hide)
     )
+    (property "JLCPCB" "C21190" (id 5) (at 33.655 50.165 0)
+      (effects (font (size 1.27 1.27)) hide)
+    )
     (pin "1")
     (pin "2")
@@
     )
     (property "MPN" "" (id 4) (at 61.595 27.94 0)
+      (effects (font (size 1.27 1.27)) hide)
+    )
+    (property "JLCPCB" "C19666" (id 5) (at 61.595 27.94 0)
       (effects (font (size 1.27 1.27)) hide)
     )
@@
       (effects (font (size 1.27 1.27)) hide)
     )
+    (property "JLCPCB" "C25804" (id 4) (at 217.805 54.61 90)
+      (effects (font (size 1.27 1.27)) hide)
+    )
     (pin "1")
     (pin "2")
@@
     )
     (property "MPN" "" (id 4) (at 33.655 69.215 0)
+      (effects (font (size 1.27 1.27)) hide)
+    )
+    (property "JLCPCB" "C21190" (id 5) (at 33.655 69.215 0)
       (effects (font (size 1.27 1.27)) hide)
     )
@@
       (effects (font (size 1.27 1.27)) hide)
     )
+    (property "JLCPCB" "C21190" (id 5) (at 33.655 118.11 0)
+      (effects (font (size 1.27 1.27)) hide)
+    )
     (pin "1")
     (pin "2")
@@
       (effects (font (size 1.27 1.27)) hide)
     )
+    (property "JLCPCB" "C25804" (id 5) (at 25.4 118.11 0)
+      (effects (font (size 1.27 1.27)) hide)
+    )
     (pin "1")
     (pin "2")
@@
       (effects (font (size 1.27 1.27)) hide)
     )
+    (property "JLCPCB" "C25804" (id 5) (at 222.885 66.04 0)
+      (effects (font (size 1.27 1.27)) hide)
+    )
     (pin "1")
     (pin "2")
@@
       (effects (font (size 1.27 1.27)) hide)
     )
+    (property "JLCPCB" "C19666" (id 5) (at 200.025 72.39 0)
+      (effects (font (size 1.27 1.27)) hide)
+    )
     (pin "1")
     (pin "2")
@@
     )
     (property "MPN" "" (id 4) (at 61.595 114.935 0)
+      (effects (font (size 1.27 1.27)) hide)
+    )
+    (property "JLCPCB" "C19666" (id 5) (at 61.595 114.935 0)
       (effects (font (size 1.27 1.27)) hide)
     )
@@
       (effects (font (size 1.27 1.27)) hide)
     )
+    (property "JLCPCB" "C14663" (id 5) (at 186.69 93.345 0)
+      (effects (font (size 1.27 1.27)) hide)
+    )
     (pin "1")
     (pin "2")
@@
       (effects (font (size 1.27 1.27)) hide)
     )
+    (property "JLCPCB" "C19666" (id 5) (at 61.595 66.04 0)
+      (effects (font (size 1.27 1.27)) hide)
+    )
     (pin "1")
     (pin "2")
@@
     )
     (property "MPN" "" (id 4) (at 61.595 46.99 0)
+      (effects (font (size 1.27 1.27)) hide)
+    )
+    (property "JLCPCB" "C19666" (id 5) (at 61.595 46.99 0)
       (effects (font (size 1.27 1.27)) hide)
     )
@@
       (effects (font (size 1.27 1.27)) hide)
     )
+    (property "JLCPCB" "C14663" (id 5) (at 73.66 177.165 0)
+      (effects (font (size 1.27 1.27)) hide)
+    )
     (pin "1")
     (pin "2")
@@
     )
     (property "MPN" "" (id 4) (at 25.4 31.115 0)
+      (effects (font (size 1.27 1.27)) hide)
+    )
+    (property "JLCPCB" "C25804" (id 5) (at 25.4 31.115 0)
       (effects (font (size 1.27 1.27)) hide)
     )
@@
       (effects (font (size 1.27 1.27)) hide)
     )
+    (property "JLCPCB" "C25804" (id 5) (at 25.4 50.165 0)
+      (effects (font (size 1.27 1.27)) hide)
+    )
     (pin "1")
     (pin "2")
@@
     )
     (property "MPN" "" (id 4) (at 25.4 88.265 0)
+      (effects (font (size 1.27 1.27)) hide)
+    )
+    (property "JLCPCB" "C25804" (id 5) (at 25.4 88.265 0)
       (effects (font (size 1.27 1.27)) hide)
     )
@@
       (effects (font (size 1.27 1.27)) hide)
     )
+    (property "JLCPCB" "C19666" (id 5) (at 198.12 34.29 0)
+      (effects (font (size 1.27 1.27)) hide)
+    )
