File: Hardware/front/controller.kicad_sch (KiCad schematic)
At the start: 22 parts

Commit message: front: minor tweaks
- added some more pull-ups on IO lines

- doubled decoupling capacitance for LEDs
Parts:
- added R: R_Small, symbol Device:R_Small
- added U: (no value), symbol Device:R_Small
- C: JLCPCB C1647 -> C1653
Connections:
- net +3V3: now also U.2
- net XOUT: now also R.2; no longer C.1, Y.3
- net ~{FLASH_CS}: now also U.1
- new net: C.1, R.1, Y.3
Changed lines of the file:
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@@
   (junction (at 35.56 91.44) (diameter 0) (color 0 0 0 0)
+  )
+  (junction (at 120.015 143.51) (diameter 0) (color 0 0 0 0)
   )
   (junction (at 29.845 192.405) (diameter 0) (color 0 0 0 0)
@@
     (stroke (width 0) (type default))
   )
-  (wire (pts (xy 88.9 128.27) (xy 101.6 128.27))
+  (wire (pts (xy 76.2 128.27) (xy 88.9 128.27))
     (stroke (width 0) (type default))
   )
@@
     (stroke (width 0) (type default))
   )
+  (wire (pts (xy 102.87 133.35) (xy 111.125 133.35))
+    (stroke (width 0) (type default))
+  )
   (wire (pts (xy 68.58 73.66) (xy 69.85 73.66))
     (stroke (width 0) (type default))
@@
     (stroke (width 0) (type default))
   )
+  (wire (pts (xy 120.015 143.51) (xy 120.015 151.765))
+    (stroke (width 0) (type default))
+  )
   (wire (pts (xy 68.58 63.5) (xy 69.85 63.5))
     (stroke (width 0) (type default))
@@
   )
   (wire (pts (xy 35.56 36.83) (xy 22.86 36.83))
+    (stroke (width 0) (type default))
+  )
+  (wire (pts (xy 125.095 151.765) (xy 137.795 151.765))
     (stroke (width 0) (type default))
   )
@@
     (effects (font (size 1.27 1.27)) (justify right bottom))
   )
+  (label "~{FLASH_CS}" (at 137.795 151.765 180) (fields_autoplaced)
+    (effects (font (size 1.27 1.27)) (justify right bottom))
+  )
   (label "STATUSLED" (at 177.8 158.75 0) (fields_autoplaced)
     (effects (font (size 1.27 1.27)) (justify left bottom))
@@
     (effects (font (size 1.27 1.27)) (justify left bottom))
   )
-  (label "XOUT" (at 97.79 133.35 0) (fields_autoplaced)
+  (label "XOUT" (at 111.125 133.35 0) (fields_autoplaced)
     (effects (font (size 1.27 1.27)) (justify right bottom))
   )
@@
     (pin "1")
   )
-  (symbol (lib_id "power:GND") (at 101.6 128.27 0) (unit 1)
+  (symbol (lib_id "power:GND") (at 76.2 128.27 0) (unit 1)
     (in_bom yes) (on_board yes)
     (default_instance (reference "#PWR") (unit 1) (value "GND") (footprint ""))
-    (property "Reference" "#PWR" (id 0) (at 101.6 134.62 0)
-      (effects (font (size 1.27 1.27)) hide)
-    )
-    (property "Value" "GND" (id 1) (at 101.6 132.715 0)
-      (effects (font (size 1.27 1.27)))
-    )
-    (property "Footprint" "" (id 2) (at 101.6 128.27 0)
-      (effects (font (size 1.27 1.27)) hide)
-    )
-    (property "Datasheet" "" (id 3) (at 101.6 128.27 0)
+    (property "Reference" "#PWR" (id 0) (at 76.2 134.62 0)
+      (effects (font (size 1.27 1.27)) hide)
+    )
+    (property "Value" "GND" (id 1) (at 76.2 132.715 0)
+      (effects (font (size 1.27 1.27)))
+    )
+    (property "Footprint" "" (id 2) (at 76.2 128.27 0)
+      (effects (font (size 1.27 1.27)) hide)
+    )
+    (property "Datasheet" "" (id 3) (at 76.2 128.27 0)
       (effects (font (size 1.27 1.27)) hide)
     )
@@
       (effects (font (size 1.27 1.27)) hide)
     )
-    (property "JLCPCB" "C1647" (id 4) (at 86.36 140.335 0)
+    (property "JLCPCB" "C1653" (id 4) (at 86.36 140.335 0)
       (effects (font (size 1.27 1.27)) hide)
     )
@@
       (effects (font (size 1.27 1.27)) hide)
     )
-    (property "JLCPCB" "C1647" (id 4) (at 91.44 140.335 0)
+    (property "JLCPCB" "C1653" (id 4) (at 91.44 140.335 0)
       (effects (font (size 1.27 1.27)) hide)
     )
@@
     (pin "1")
   )
+  (symbol (lib_id "Device:R_Small") (at 100.33 133.35 90) (unit 1)
+    (in_bom yes) (on_board yes) (fields_autoplaced)
+    (default_instance (reference "R") (unit 1) (value "R_Small") (footprint ""))
+    (property "Reference" "R" (id 0) (at 100.33 128.27 90)
+      (effects (font (size 1.27 1.27)))
+    )
+    (property "Value" "R_Small" (id 1) (at 100.33 130.81 90)
+      (effects (font (size 1.27 1.27)))
+    )
+    (property "Footprint" "" (id 2) (at 100.33 133.35 0)
+      (effects (font (size 1.27 1.27)) hide)
+    )
+    (property "Datasheet" "~" (id 3) (at 100.33 133.35 0)
+      (effects (font (size 1.27 1.27)) hide)
+    )
+    (property "JLCPCB" "C21190" (id 4) (at 100.33 133.35 90)
+      (effects (font (size 1.27 1.27)) hide)
+    )
+    (pin "1")
+    (pin "2")
+  )
   (symbol (lib_id "Device:R_Small") (at 122.555 127 270) (mirror x) (unit 1)
     (in_bom yes) (on_board yes)
@@
     (pin "1")
   )
+  (symbol (lib_id "Device:R_Small") (at 122.555 151.765 270) (mirror x) (unit 1)
+    (in_bom yes) (on_board yes)
+    (default_instance (reference "U") (unit 1) (value "") (footprint ""))
+    (property "Reference" "U" (id 0) (at 122.555 146.685 90)
+      (effects (font (size 1.27 1.27)))
+    )
+    (property "Value" "" (id 1) (at 122.555 149.225 90)
+      (effects (font (size 1.27 1.27)))
+    )
+    (property "Footprint" "" (id 2) (at 122.555 151.765 0)
+      (effects (font (size 1.27 1.27)) hide)
+    )
+    (property "Datasheet" "~" (id 3) (at 122.555 151.765 0)
+      (effects (font (size 1.27 1.27)) hide)
+    )
+    (property "MPN" "" (id 4) (at 122.555 151.765 90)
+      (effects (font (size 1.27 1.27)) hide)
+    )
+    (property "JLCPCB" "C25804" (id 5) (at 122.555 151.765 90)
+      (effects (font (size 1.27 1.27)) hide)
+    )
+    (pin "1")
+    (pin "2")
+  )
   (symbol (lib_id "power:GND") (at 88.9 142.875 0) (unit 1)

Commit message: Minor tweaks for RTC, IO section
Parts:
- removed TP (x2): TestPoint, symbol Connector:TestPoint
- removed U (x2): (no value), symbol Device:R_Small
Connections:
- net I²C_SCL: no longer names the net of U.30 (GPIO19)
- net I²C_SDA: no longer names the net of U.29 (GPIO18)
- no-connect marks 11 -> 13
Changed lines of the file:
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@@
   (junction (at 35.56 91.44) (diameter 0) (color 0 0 0 0)
   )
-  (junction (at 120.015 143.51) (diameter 0) (color 0 0 0 0)
-  )
   (junction (at 29.845 192.405) (diameter 0) (color 0 0 0 0)
   )
@@
   )
   (junction (at 25.4 147.32) (diameter 0) (color 0 0 0 0)
-  )
-  (junction (at 120.015 135.255) (diameter 0) (color 0 0 0 0)
   )
   (junction (at 35.56 120.65) (diameter 0) (color 0 0 0 0)
@@
   (no_connect (at 68.58 22.86))
   (no_connect (at 68.58 55.88))
+  (no_connect (at 68.58 68.58))
   (no_connect (at 42.545 182.245))
   (no_connect (at 68.58 58.42))
+  (no_connect (at 68.58 71.12))
   (wire (pts (xy 68.58 50.8) (xy 69.85 50.8))
     (stroke (width 0) (type default))
@@
     (stroke (width 0) (type default))
   )
-  (wire (pts (xy 125.095 135.255) (xy 126.365 135.255))
-    (stroke (width 0) (type default))
-  )
   (wire (pts (xy 68.58 91.44) (xy 69.85 91.44))
     (stroke (width 0) (type default))
@@
     (stroke (width 0) (type default))
   )
-  (wire (pts (xy 120.015 143.51) (xy 120.015 151.765))
-    (stroke (width 0) (type default))
-  )
   (wire (pts (xy 68.58 63.5) (xy 69.85 63.5))
     (stroke (width 0) (type default))
@@
     (stroke (width 0) (type default))
   )
-  (wire (pts (xy 125.095 143.51) (xy 126.365 143.51))
-    (stroke (width 0) (type default))
-  )
   (wire (pts (xy 35.56 81.28) (xy 35.56 83.82))
     (stroke (width 0) (type default))
@@
     (stroke (width 0) (type default))
   )
-  (wire (pts (xy 158.75 135.255) (xy 160.02 135.255))
-    (stroke (width 0) (type default))
-  )
   (wire (pts (xy 42.545 174.625) (xy 55.245 174.625))
     (stroke (width 0) (type default))
@@
     (stroke (width 0) (type default))
   )
-  (wire (pts (xy 68.58 71.12) (xy 69.85 71.12))
-    (stroke (width 0) (type default))
-  )
   (wire (pts (xy 25.4 120.65) (xy 35.56 120.65))
     (stroke (width 0) (type default))
@@
     (stroke (width 0) (type default))
   )
-  (wire (pts (xy 120.015 127) (xy 120.015 135.255))
-    (stroke (width 0) (type default))
-  )
-  (wire (pts (xy 68.58 68.58) (xy 69.85 68.58))
+  (wire (pts (xy 120.015 127) (xy 120.015 151.765))
     (stroke (width 0) (type default))
   )
@@
   )
   (wire (pts (xy 35.56 41.91) (xy 22.86 41.91))
-    (stroke (width 0) (type default))
-  )
-  (wire (pts (xy 158.75 127) (xy 160.02 127))
-    (stroke (width 0) (type default))
-  )
-  (wire (pts (xy 120.015 135.255) (xy 120.015 143.51))
     (stroke (width 0) (type default))
   )
@@
     (effects (font (size 1.27 1.27)) (justify left bottom))
   )
-  (hierarchical_label "I²C_SCL" (shape bidirectional) (at 126.365 135.255 0) (fields_autoplaced)
-    (effects (font (size 1.27 1.27)) (justify left))
-  )
   (hierarchical_label "SW_MENU" (shape input) (at 69.85 50.8 0) (fields_autoplaced)
     (effects (font (size 1.27 1.27)) (justify left))
@@
     (effects (font (size 1.27 1.27)) (justify left))
   )
-  (hierarchical_label "I²C_SDA" (shape bidirectional) (at 160.02 135.255 0) (fields_autoplaced)
-    (effects (font (size 1.27 1.27)) (justify left))
-  )
   (hierarchical_label "SW_MODE_CV" (shape input) (at 69.85 38.1 0) (fields_autoplaced)
     (effects (font (size 1.27 1.27)) (justify left))
   )
-  (hierarchical_label "I²C_SDA" (shape bidirectional) (at 69.85 68.58 0) (fields_autoplaced)
-    (effects (font (size 1.27 1.27)) (justify left))
-  )
-  (hierarchical_label "I²C_SCL" (shape bidirectional) (at 69.85 71.12 0) (fields_autoplaced)
-    (effects (font (size 1.27 1.27)) (justify left))
-  )
   (hierarchical_label "HOST_I²C_SDA" (shape bidirectional) (at 69.85 83.82 0) (fields_autoplaced)
     (effects (font (size 1.27 1.27)) (justify left))
   )
   (hierarchical_label "SW_MODE_EXT" (shape input) (at 69.85 40.64 0) (fields_autoplaced)
-    (effects (font (size 1.27 1.27)) (justify left))
-  )
-  (hierarchical_label "I²C_SDA" (shape bidirectional) (at 126.365 143.51 0) (fields_autoplaced)
-    (effects (font (size 1.27 1.27)) (justify left))
-  )
-  (hierarchical_label "I²C_SCL" (shape bidirectional) (at 160.02 127 0) (fields_autoplaced)
     (effects (font (size 1.27 1.27)) (justify left))
   )
@@
     (pin "1")
     (pin "2")
-  )
-  (symbol (lib_id "Connector:TestPoint") (at 158.75 127 90) (unit 1)
-    (in_bom no) (on_board yes) (fields_autoplaced)
-    (default_instance (reference "TP") (unit 1) (value "TestPoint") (footprint ""))
-    (property "Reference" "TP" (id 0) (at 155.448 121.92 90)
-      (effects (font (size 1.27 1.27)))
-    )
-    (property "Value" "TestPoint" (id 1) (at 155.448 124.46 90)
-      (effects (font (size 1.27 1.27)))
-    )
-    (property "Footprint" "" (id 2) (at 158.75 121.92 0)
-      (effects (font (size 1.27 1.27)) hide)
-    )
-    (property "Datasheet" "~" (id 3) (at 158.75 121.92 0)
-      (effects (font (size 1.27 1.27)) hide)
-    )
-    (pin "1")
   )
   (symbol (lib_id "power:+1V1") (at 25.4 142.24 0) (unit 1)
@@
     (pin "2")
   )
-  (symbol (lib_id "Device:R_Small") (at 122.555 135.255 270) (mirror x) (unit 1)
-    (in_bom yes) (on_board yes)
-    (default_instance (reference "U") (unit 1) (value "") (footprint ""))
-    (property "Reference" "U" (id 0) (at 122.555 130.175 90)
-      (effects (font (size 1.27 1.27)))
-    )
-    (property "Value" "" (id 1) (at 122.555 132.715 90)
-      (effects (font (size 1.27 1.27)))
-    )
-    (property "Footprint" "" (id 2) (at 122.555 135.255 0)
-      (effects (font (size 1.27 1.27)) hide)
-    )
-    (property "Datasheet" "~" (id 3) (at 122.555 135.255 0)
-      (effects (font (size 1.27 1.27)) hide)
-    )
-    (property "MPN" "" (id 4) (at 122.555 135.255 90)
-      (effects (font (size 1.27 1.27)) hide)
-    )
-    (property "JLCPCB" "C4190" (id 5) (at 122.555 135.255 90)
-      (effects (font (size 1.27 1.27)) hide)
-    )
-    (pin "1")
-    (pin "2")
-  )
   (symbol (lib_id "power:+1V1") (at 35.56 91.44 90) (unit 1)
     (in_bom yes) (on_board yes)
@@
     (pin "4")
   )
-  (symbol (lib_id "Device:R_Small") (at 122.555 143.51 270) (mirror x) (unit 1)
-    (in_bom yes) (on_board yes)
-    (default_instance (reference "U") (unit 1) (value "") (footprint ""))
-    (property "Reference" "U" (id 0) (at 122.555 138.43 90)
-      (effects (font (size 1.27 1.27)))
-    )
-    (property "Value" "" (id 1) (at 122.555 140.97 90)
-      (effects (font (size 1.27 1.27)))
-    )
-    (property "Footprint" "" (id 2) (at 122.555 143.51 0)
-      (effects (font (size 1.27 1.27)) hide)
-    )
-    (property "Datasheet" "~" (id 3) (at 122.555 143.51 0)
-      (effects (font (size 1.27 1.27)) hide)
-    )
-    (property "MPN" "" (id 4) (at 122.555 143.51 90)
-      (effects (font (size 1.27 1.27)) hide)
-    )
-    (property "JLCPCB" "C4190" (id 5) (at 122.555 143.51 90)
-      (effects (font (size 1.27 1.27)) hide)
-    )
-    (pin "1")
-    (pin "2")
-  )
   (symbol (lib_id "power:GND") (at 19.685 58.42 0) (unit 1)
     (in_bom yes) (on_board yes)
@@
     (pin "2")
   )
-  (symbol (lib_id "Connector:TestPoint") (at 158.75 135.255 90) (unit 1)
-    (in_bom no) (on_board yes) (fields_autoplaced)
-    (default_instance (reference "TP") (unit 1) (value "TestPoint") (footprint ""))
-    (property "Reference" "TP" (id 0) (at 155.448 130.81 90)
-      (effects (font (size 1.27 1.27)))
-    )
-    (property "Value" "TestPoint" (id 1) (at 155.448 133.35 90)
-      (effects (font (size 1.27 1.27)))
-    )
-    (property "Footprint" "" (id 2) (at 158.75 130.175 0)
-      (effects (font (size 1.27 1.27)) hide)
-    )
-    (property "Datasheet" "~" (id 3) (at 158.75 130.175 0)
-      (effects (font (size 1.27 1.27)) hide)
-    )
-    (pin "1")
-  )
   (symbol (lib_id "Device:C_Small") (at 35.56 123.19 0) (mirror y) (unit 1)
